File: KiCad/OTO_NO_ITA/mcu.kicad_sch (KiCad schematic)
At the start: 1 part, among them U1 STM32H7S3Z8Tx

Commit message: Updated schematics.
Parts:
- added C39, C44, C45, C46, C47, C48, C49, C50, C51, C52, C53, C54, C55, C56, C57, C58, C59, C60, C64: 100nF, symbol Device:C
- added C40: 100nF, Capacitor_SMD:C_0402_1005Metric, symbol Device:C
- added C41, C42, C43, C66: 2.2uF, symbol Device:C
- added C61, C62: 4.7uF, symbol Device:C
- added C63, C65: 1uF, symbol Device:C
- added R10, R11, R12: 10k, symbol Device:R
- added R13: 33R, Resistor_SMD:R_0402_1005Metric, symbol Device:R
- added SW2: SW_MEC_5G, symbol My_Parts:SW_MEC_5G
- added U5: MX25UW25645GXDI00, symbol My_Parts:MX25UW25645GXDI00
- added X2: 24MHz, symbol Oscillator:SG-8002CE
Connections:
- net 3V3: now reaches U1.100 (VDD)
- net 3V3: now also U1.108 (VDD), U1.115 (VDD50USB), U1.116 (VDD33USB), U1.123 (VDD), U1.133 (VDD), U1.139 (VDD), U1.17 (VDD), U1.23 (VREFM), U1.25 (VDDA), U1.3 (VBAT), U1.31 (VDD), U1.41 (VDD), U1.69 (VDD), U1.7 (VDD), U1.81 (VDD), U1.88 (VDD), C40.2, C45.2, C46.2, C47.2, C48.2, C49.2, C50.2, C51.2, C52.2, C53.2, C54.2, C55.2, C56.2, C61.2, C63.2, C64.2, C65.2, X2.4 (Vcc)
- net GND: now reaches U1.107 (VSS), U1.132 (VSS), U1.138 (VSS), U1.16 (VSS), U1.30 (VSS), U1.42 (VSS), U1.46 (VSS), U1.50 (VSS), U1.56 (VSS), U1.62 (VSS), U1.70 (VSS), U1.8 (VSS), U1.80 (VSS), U1.89 (VSS), U1.99 (VSS)
- net GND: now also U1.117 (VSSUSB), U1.22 (VSSA), U1.24 (VREFP), C39.1, C40.1, C41.1, C42.1, C43.1, C44.1, C45.1, C46.1, C47.1, C48.1, C49.1, C50.1, C51.1, C52.1, C53.1, C54.1, C55.1, C56.1, C57.1, C58.1, C59.1, C60.1, C61.1, C62.1, C63.1, C64.1, C65.1, C66.1, R10.1, SW2.1 (A), X2.2 (GND)
- net UCPD_CC1: now reaches U1.111 (PM0)
- net UCPD_CC2: now reaches U1.112 (PM1)
- net USB_HS_D-: now reaches U1.118 (PM5)
- net USB_HS_D+: now reaches U1.119 (PM6)
- net MCU_DVDD: now reaches U1.120 (DVDD)
- net MCU_DVDD: now also U1.137 (VCAP4), U1.43 (VCAP1), U1.79 (VCAP2), U1.98 (VCAP3), C41.2, C42.2, C43.2, C44.2, C66.2
- net UCPD_INT: now reaches U1.121 (PM8)
- net UCPD_PWR_EN: now reaches U1.122 (PM9)
- net at U1.128 (BOOT0): now also R10.2
- net at U1.13 (PH0): now also R13.2
- net DEBUG_SWO: now reaches U1.134 (PB3(JTDO)
- net NRST: now reaches U1.15 (NRST)
- net NRST: now also C39.2, SW2.3 (B), U5.A4 (RESET)
- net 1V8: now reaches U1.45 (VDDXSPI1)
- net 1V8: now also U1.51 (VDDXSPI1), U1.57 (VDDXSPI1), U1.63 (VDDXSPI1), C57.2, C58.2, C59.2, C60.2, C62.2, R11.1, R12.2
- net at U1.47 (PP4): now also U5.D5 (SIO4)
- net at U1.48 (PP2): now also U5.C4 (SIO2)
- net at U1.49 (PP3): now also U5.D4 (SIO3)
- net at U1.53 (PO4): now also U5.B2 (SCLK)
- net at U1.54 (PP5): now also U5.E3 (SIO5)
- net at U1.55 (PP0): now also U5.D3 (SIO0)
- net at U1.58 (PP6): now also U5.E2 (SIO6)
- net at U1.59 (PO2): now also U5.C3 (DQS)
- net at U1.60 (PP7): now also U5.E1 (SIO7)
- net at U1.61 (PP1): now also U5.D2 (SIO1)
- net at U1.64 (PO0): now also R12.1, U5.C2 (CS)
- net I2S_CLKIN: now reaches U1.87 (PC9)
- net DEBUG_SWDIO: now reaches U1.95 (PA13(JTMS)
- net DEBUG_SWCLK: now reaches U1.96 (PA14(JTCK)
- new net: R13.1, X2.3 (OUT)
- new net: R11.2, U5.A5 (ECS)
- no-connect marks 0 -> 1
Other:
- moved on the sheet: U1

Commit message: Updated schematics.
Connections:
- net SAI_FS: now reaches U1.10 (PE4)
- net SAI_SCK: now reaches U1.11 (PE5)
- net SAI_DATA_OUT: now reaches U1.12 (PE6)
- net SPI5_SS: now reaches U1.124 (PM12)
- net SPI5_SCLK: now reaches U1.125 (PM11)
- net SPI5_MISO: now reaches U1.126 (PM14)
- net SPI5_MOSI: now reaches U1.127 (PM13)
- net ADC1_IN10: now reaches U1.18 (PC0)
- net ADC1_IN11: now reaches U1.19 (PC1)
- net ADC1_IN12: now reaches U1.20 (PC2)
- net ADC1_IN13: now reaches U1.21 (PC3)
- net ADC1_IN0: now reaches U1.26 (PA0)
- net ADC1_IN1: now reaches U1.27 (PA1)
- net ADC1_IN14: now reaches U1.28 (PA2)
- net ADC1_IN15: now reaches U1.29 (PA3)
- net ADC1_IN18: now reaches U1.32 (PA4)
- net ADC1_IN3: now reaches U1.34 (PA6)
- net ADC1_IN7: now reaches U1.35 (PA7)
- net ADC1_IN4: now reaches U1.36 (PC4)
- net ADC1_IN8: now reaches U1.37 (PC5)
- net ADC1_IN9: now reaches U1.38 (PB0)
- net ADC1_IN5: now reaches U1.39 (PB1)
- net I2C2_SCL: now reaches U1.73 (PB10)
- net I2C2_SDA: now reaches U1.74 (PB11)
- net SAI_DATA_IN: now reaches U1.9 (PE3)
Other:
- moved on the sheet: C41, C42, C43, C66

Commit message: Updated schematics.
Parts:
- added C67, C68, C69: 100nF, Capacitor_SMD:C_0402_1005Metric, symbol Device:C
- added C70, C71, C72: 4.7uF, Capacitor_SMD:C_0402_1005Metric, symbol Device:C
- added J2, J3, J8: Conn_01x07, My_Parts:PinHeader_1x07_P2.54mm_Vertical, symbol Connector_Generic:Conn_01x07
Connections:
- net 1V8: now also U5.B4 (VCC), U5.D1 (VCCQ), U5.E4 (VCCQ), C67.2, C68.2, C69.2, C70.2, C71.2, C72.2
- net 3V3: now also J2.1 (Pin_1), J3.1 (Pin_1), J8.1 (Pin_1)
- net ADC1_IN0: now also J2.2 (Pin_2)
- net ADC1_IN1: now also J2.3 (Pin_3)
- net ADC1_IN10: now also J3.5 (Pin_5)
- net ADC1_IN11: now also J3.6 (Pin_6)
- net ADC1_IN12: now also J8.2 (Pin_2)
- net ADC1_IN13: now also J8.3 (Pin_3)
- net ADC1_IN14: now also J8.4 (Pin_4)
- net ADC1_IN15: now also J8.5 (Pin_5)
- net ADC1_IN18: now also J8.6 (Pin_6)
- net ADC1_IN3: now also J2.4 (Pin_4)
- net ADC1_IN4: now also J2.5 (Pin_5)
- net ADC1_IN5: now also J2.6 (Pin_6)
- net ADC1_IN7: now also J3.2 (Pin_2)
- net ADC1_IN8: now also J3.3 (Pin_3)
- net ADC1_IN9: now also J3.4 (Pin_4)
- net GND: now also U5.B3 (GND), U5.C1 (VSSQ), U5.E5 (VSSQ), C67.1, C68.1, C69.1, C70.1, C71.1, C72.1, J2.7 (Pin_7), J3.7 (Pin_7), J8.7 (Pin_7)
- net DSP_RESET: now reaches U1.14 (PH1)
- no-connect marks 1 -> 8
Other:
- note added: "11 ports"
- note added: "16 ports"
- note added: "6 ports"
- note added: "7 ports"
- moved on the sheet: R11, R12, U5

Commit message: Assigned footprint.
Parts:
- C39, C44, C45, C46, C47, C48, C49, C50, C51, C52, C53, C54, C55, C56, C57, C58, C59, C60, C64: footprint (none) -> Capacitor_SMD:C_0201_0603Metric
- C40: footprint Capacitor_SMD:C_0402_1005Metric -> Capacitor_SMD:C_0201_0603Metric
- C41, C42, C43, C61, C62, C63, C65, C66: footprint (none) -> Capacitor_SMD:C_0402_1005Metric
- R10, R11, R12: footprint (none) -> Resistor_SMD:R_0201_0603Metric
- R13: footprint Resistor_SMD:R_0402_1005Metric -> Resistor_SMD:R_0201_0603Metric
- SW2: footprint (none) -> My_Parts:SKRPABE010
- U5: footprint (none) -> My_Parts:BGA24C100P5X5_800X600X120
- X2: footprint (none) -> Oscillator:Oscillator_SMD_SeikoEpson_SG210-4Pin_2.5x2.0mm
Other:
- moved on the sheet: C40, C41, C42, C43, C66, R13, X2

Commit message: Updated schematics.
Parts:
- removed SW2: SW_MEC_5G, My_Parts:SKRPABE010, symbol My_Parts:SW_MEC_5G
- added C32: 100nF, Capacitor_SMD:C_0201_0603Metric, symbol Device:C
- added J4: 15910060, My_Parts:Molex_15910060, symbol Connector_Generic:Conn_02x03_Odd_Even
- added SW1: SKRPABE010, My_Parts:SKRPABE010, symbol Switch:SW_MEC_5E
- renumbered C63 to C1, C50 to C10, C51 to C11, C52 to C12, C53 to C13, C54 to C14, C55 to C15, C56 to C16, C61 to C17, C39 to C18, C71 to C19, C44 to C2, C68 to C20, C65 to C21, C64 to C22, C72 to C23, C69 to C24, C57 to C25, C58 to C26, C59 to C27, C60 to C28, C62 to C29, C70 to C3, C40 to C30, C41 to C31, C42 to C33, C43 to C34, C66 to C35, C67 to C4, C45 to C5, C46 to C6, C47 to C7, C48 to C8, C49 to C9, J2 to J1, J3 to J2, J8 to J3, R10 to R1, R12 to R2, R11 to R3, R13 to R4, U5 to U1, U1 to U2, X2 to X1
Connections:
- net 3V3: now also C32.2, J4.5 (Pin_5)
- net DEBUG_SWCLK: now also J4.4 (Pin_4)
- net DEBUG_SWDIO: now also J4.6 (Pin_6)
- net GND: now also C32.1, J4.1 (Pin_1), J4.3 (Pin_3), SW1.1, SW1.2
- net NRST: now also J4.2 (Pin_2), SW1.3 (K), SW1.4 (A)
- net UCPD_ISENSE: now reaches U2.33 (PA5)
- net DEBUG_SWO: no longer names the net of U2.134 (PB3(JTDO)
Other:
- note added: "12 ports"
- note added: "3 ports"
- note removed: "11 ports"
- note removed: "7 ports"

Commit message: Added USER_SW.
Parts:
- added C69: 100nF, Capacitor_SMD:C_0201_0603Metric, symbol Device:C
- added SW3: SKRPABE010, My_Parts:SKRPABE010, symbol Switch:SW_MEC_5E
Connections:
- net GND: now also C69.1, SW3.1, SW3.2
- net USER_SW1: now reaches U2.113 (PM2)
- net USER_SW1: now also C69.2, SW3.3 (K), SW3.4 (A)
- no-connect marks 8 -> 7

Commit message: Re-annotation.
Parts:
- removed J1, J2, J3: Conn_01x07, My_Parts:PinHeader_1x07_P2.54mm_Vertical, symbol Connector_Generic:Conn_01x07
- added C17, C38: 100nF, Capacitor_SMD:C_0201_0603Metric, symbol Device:C
- added D1, D2, D3, D4: LED, LED_SMD:LED_0603_1608Metric, symbol Device:LED
- added J1: Conn_02x09_Odd_Even, Connector_PinHeader_2.54mm:PinHeader_2x09_P2.54mm_Vertical, symbol Connector_Generic:Conn_02x09_Odd_Even
- added J2: Conn_02x12_Odd_Even, Connector_PinHeader_2.54mm:PinHeader_2x12_P2.54mm_Vertical, symbol Connector_Generic:Conn_02x12_Odd_Even
- added J3: Conn_02x13_Odd_Even, Connector_PinHeader_2.54mm:PinHeader_2x13_P2.54mm_Vertical, symbol Connector_Generic:Conn_02x13_Odd_Even
- added R5, R6, R7, R8: 1k, Resistor_SMD:R_0201_0603Metric, symbol Device:R
- added SW3: SKRPABE010, My_Parts:SKRPABE010, symbol Switch:SW_MEC_5E
- J4: footprint My_Parts:Molex_15910060 -> Connector_PinHeader_2.54mm:PinHeader_2x03_P2.54mm_Vertical
- renumbered C17 to C18, C18 to C19, C19 to C20, C20 to C21, C21 to C22, C22 to C23, C23 to C24, C24 to C25, C25 to C26, C26 to C27, C27 to C28, C28 to C29, C29 to C30, C30 to C31, C31 to C32, C32 to C34, C34 to C35, C35 to C36, C69 to C37, SW3 to SW2
Connections:
- net 3V3: now also C17.2, J1.1 (Pin_1), J1.2 (Pin_2), J2.1 (Pin_1), J2.2 (Pin_2), J3.1 (Pin_1), J3.2 (Pin_2), R5.1
- net ADC1_IN0: now also J1.3 (Pin_3)
- net ADC1_IN10: now also J1.9 (Pin_9)
- net ADC1_IN12: now also J1.11 (Pin_11)
- net ADC1_IN13: now also J1.13 (Pin_13)
- net ADC1_IN15: now also J1.15 (Pin_15)
- net ADC1_IN3: now also J1.5 (Pin_5)
- net ADC1_IN5: now also J1.7 (Pin_7)
- net GND: now also C17.1, C38.1, D1.1 (K), D2.1 (K), D3.1 (K), D4.1 (K), J1.17 (Pin_17), J1.18 (Pin_18), J2.21 (Pin_21), J2.23 (Pin_23), J2.24 (Pin_24), J3.24 (Pin_24), J3.25 (Pin_25), J3.26 (Pin_26), SW3.1, SW3.2
- net I2C2_SCL: now also U2.90 (PA8); no longer U2.73 (PB10)
- net I2C2_SDA: now also U2.91 (PA9); no longer U2.74 (PB11)
- net USER_SW1: now also U2.44 (PO1); no longer U2.113 (PM2)
- net SDMMC2_D4: now reaches U2.1 (PB8)
- net SDMMC2_D4: now also J3.16 (Pin_16)
- net I2S3_CK: now reaches U2.101 (PC10)
- net I2S3_CK: now also J2.11 (Pin_11)
- net I2S3_SDI: now reaches U2.102 (PC11)
- net I2S3_SDI: now also J2.17 (Pin_17)
- net PD0: now reaches U2.104 (PD0)
- net PD0: now also J2.4 (Pin_4)
- net PD1: now reaches U2.105 (PD1)
- net PD1: now also J2.6 (Pin_6)
- net PD2: now reaches U2.106 (PD2)
- net PD2: now also J2.8 (Pin_8)
- net PD3: now reaches U2.109 (PD3)
- net PD3: now also J2.10 (Pin_10)
- net ETH_RMII_INTN: now reaches U2.110 (PD4)
- net ETH_RMII_INTN: now also J3.19 (Pin_19)
- net PD5: now reaches U2.129 (PD5)
- net PD5: now also J2.12 (Pin_12)
- net SDMMC2_CK: now reaches U2.130 (PD6)
- net SDMMC2_CK: now also J3.4 (Pin_4)
- net SDMMC2_CMD: now reaches U2.131 (PD7)
- net SDMMC2_CMD: now also J3.6 (Pin_6)
- net SDMMC2_D2: now reaches U2.134 (PB3(JTDO)
- net SDMMC2_D2: now also J3.12 (Pin_12)
- net SDMMC2_D3: now reaches U2.135 (PB4(NJTRST))
- net SDMMC2_D3: now also J3.14 (Pin_14)
- net PB5: now reaches U2.136 (PB5)
- net PE0: now reaches U2.140 (PE0)
- net PE0: now also J2.20 (Pin_20)
- net PE1: now reaches U2.141 (PE1)
- net PE1: now also J2.19 (Pin_19)
- net PE2: now reaches U2.142 (PE2)
- net PE2: now also J2.22 (Pin_22)
- net LPUART1_TX: now reaches U2.143 (PB6)
- net LPUART1_TX: now also J2.3 (Pin_3)
- net ETH_RMII_TXD1: now reaches U2.144 (PB7)
- net ETH_RMII_TXD1: now also J3.11 (Pin_11)
- net SDMMC2_D5: now reaches U2.2 (PB9)
- net SDMMC2_D5: now also J3.18 (Pin_18)
- net LED0: now reaches U2.4 (PC13)
- net LED0: now also R6.1
- net I2S3_SDO: now reaches U2.40 (PB2)
- net I2S3_SDO: now also J2.15 (Pin_15)
- net LED1: now reaches U2.5 (PC14)
- net LED1: now also R7.1
- net USER_SW2: now reaches U2.52 (PO5)
- net USER_SW2: now also C38.2, SW3.3 (K), SW3.4 (A)
- net LED2: now reaches U2.6 (PC15)
- net LED2: now also R8.1
- net USART3_TX: now reaches U2.65 (PD8)
- net USART3_TX: now also J1.4 (Pin_4)
- net USART3_RX: now reaches U2.66 (PD9)
- net USART3_RX: now also J1.6 (Pin_6)
- net USART3_CK: now reaches U2.67 (PD10)
- net USART3_CK: now also J1.8 (Pin_8)
- net USART3_CTS: now reaches U2.68 (PD11)
- net USART3_CTS: now also J1.10 (Pin_10)
- net USART3_RTS: now reaches U2.71 (PD12)
- net USART3_RTS: now also J1.12 (Pin_12)
- net PD13: now reaches U2.72 (PD13)
- net PD13: now also J2.14 (Pin_14)
- net FDCAN2_RX: now reaches U2.75 (PB12)
- net FDCAN2_RX: now also J1.14 (Pin_14)
- net FDCAN2_TX: now reaches U2.76 (PB13)
- net FDCAN2_TX: now also J1.16 (Pin_16)
- net SDMMC2_D0: now reaches U2.77 (PB14)
- net SDMMC2_D0: now also J3.8 (Pin_8)
- net SDMMC2_D1: now reaches U2.78 (PB15)
- net SDMMC2_D1: now also J3.10 (Pin_10)
- net PD14: now reaches U2.82 (PD14)
- net PD14: now also J2.16 (Pin_16)
- net PD15: now reaches U2.83 (PD15)
- net PD15: now also J2.18 (Pin_18)
- net SDMMC2_D6: now reaches U2.84 (PC6)
- net SDMMC2_D6: now also J3.20 (Pin_20)
- net SDMMC2_D7: now reaches U2.85 (PC7)
- net SDMMC2_D7: now also J3.22 (Pin_22)
- net LPUART1_RX: now reaches U2.92 (PA10)
- net LPUART1_RX: now also J2.5 (Pin_5)
- net LPUART1_CTS: now reaches U2.93 (PA11)
- net LPUART1_CTS: now also J2.7 (Pin_7)
- net LPUART1_RTS: now reaches U2.94 (PA12)
- net LPUART1_RTS: now also J2.9 (Pin_9)
- net I2S3_WS: now reaches U2.97 (PA15(JTDI))
- net I2S3_WS: now also J2.13 (Pin_13)
- net ADC1_IN1 renamed ETH_RMII_REF_CLK
- net ETH_RMII_REF_CLK: now also J3.3 (Pin_3)
- net ADC1_IN11 renamed ETH_MDC
- net ETH_MDC: now also J3.13 (Pin_13)
- net ADC1_IN14 renamed ETH_MDIO
- net ETH_MDIO: now also J3.5 (Pin_5)
- net ADC1_IN4 renamed ETH_RMII_RXD0
- net ETH_RMII_RXD0: now also J3.15 (Pin_15)
- net ADC1_IN7 renamed ETH_RMII_CRS_DV
- net ETH_RMII_CRS_DV: now also J3.7 (Pin_7)
- net ADC1_IN8 renamed ETH_RMII_RXD1
- net ETH_RMII_RXD1: now also J3.17 (Pin_17)
- net ADC1_IN9 renamed ETH_RMII_TXD0
- net ETH_RMII_TXD0: now also J3.9 (Pin_9)
- new net: D3.2 (A), R7.2
- new net: D1.2 (A), R5.2
- new net: D4.2 (A), R8.2
- new net: D2.2 (A), R6.2
- new net ETH_MII_RX_ER: J3.23 (Pin_23), U2.73 (PB10)
- new net ETH_RMII_TX_EN: J3.21 (Pin_21), U2.74 (PB11)
- no-connect marks 7 -> 5
Other:
- note removed: "12 ports"
- note removed: "16 ports"
- note removed: "3 ports"
- note removed: "6 ports"
- moved on the sheet: C18, C34, C37, J4, SW2

Commit message: Change the order of IO assignment to pin headers.
Parts:
- removed J1: Conn_02x09_Odd_Even, Connector_PinHeader_2.54mm:PinHeader_2x09_P2.54mm_Vertical, symbol Connector_Generic:Conn_02x09_Odd_Even
- removed J2: Conn_02x12_Odd_Even, Connector_PinHeader_2.54mm:PinHeader_2x12_P2.54mm_Vertical, symbol Connector_Generic:Conn_02x12_Odd_Even
- added J1: Conn_02x10_Odd_Even, Connector_PinHeader_2.54mm:PinHeader_2x10_P2.54mm_Vertical, symbol Connector_Generic:Conn_02x10_Odd_Even
- added J2: Conn_02x06_Odd_Even, Connector_PinHeader_2.54mm:PinHeader_2x06_P2.54mm_Vertical, symbol Connector_Generic:Conn_02x06_Odd_Even
Connections:
- net PD0 is gone; now on net LED2: U2.104 (PD0)
- net PD1 is gone; now on net LED1: U2.105 (PD1)
- net PD14 is gone; now on net USER_SW2: U2.82 (PD14)
- net PD15 is gone; now on net USER_SW1: U2.83 (PD15)
- net PD2 is gone; now on net LED0: U2.106 (PD2)
- net 3V3: now also J1.1 (Pin_1), J1.2 (Pin_2), J2.1 (Pin_1), J2.2 (Pin_2)
- net ADC1_IN0: now also J2.3 (Pin_3)
- net ADC1_IN10: now also J2.6 (Pin_6)
- net ADC1_IN12: now also J2.7 (Pin_7)
- net ADC1_IN13: now also J2.8 (Pin_8)
- net ADC1_IN15: now also J2.9 (Pin_9)
- net ADC1_IN3: now also J2.4 (Pin_4)
- net ADC1_IN5: now also J2.5 (Pin_5)
- net FDCAN2_RX: now also J1.14 (Pin_14)
- net FDCAN2_TX: now also J1.16 (Pin_16)
- net GND: now also J1.19 (Pin_19), J2.10 (Pin_10), J2.11 (Pin_11), J2.12 (Pin_12)
- net I2C2_SCL: now also J1.18 (Pin_18)
- net I2C2_SDA: now also J1.20 (Pin_20)
- net I2S3_CK: now also J1.11 (Pin_11)
- net I2S3_SDI: now also J1.17 (Pin_17)
- net I2S3_SDO: now also J1.15 (Pin_15)
- net I2S3_WS: now also J1.13 (Pin_13)
- net LED0: no longer U2.4 (PC13)
- net LED1: no longer U2.5 (PC14)
- net LED2: no longer U2.6 (PC15)
- net LPUART1_CTS: now also J1.7 (Pin_7)
- net LPUART1_RTS: now also J1.9 (Pin_9)
- net LPUART1_RX: now also J1.5 (Pin_5)
- net LPUART1_TX: now also J1.3 (Pin_3)
- net USART3_CK: now also J1.8 (Pin_8)
- net USART3_CTS: now also J1.10 (Pin_10)
- net USART3_RTS: now also J1.12 (Pin_12)
- net USART3_RX: now also J1.6 (Pin_6)
- net USART3_TX: now also J1.4 (Pin_4)
- net USER_SW1: no longer U2.44 (PO1)
- net USER_SW2: no longer U2.52 (PO5)
- net PD13: no longer names the net of U2.72 (PD13)
- net PD3: no longer names the net of U2.109 (PD3)
- net PD5: no longer names the net of U2.129 (PD5)
- net PE0: no longer names the net of U2.140 (PE0)
- net PE1: no longer names the net of U2.141 (PE1)
- net PE2: no longer names the net of U2.142 (PE2)
- new net PO1: U2.44 (PO1)
- new net PO5: U2.52 (PO5)
- no-connect marks 5 -> 14
