File: KiCad/OTO_NO_ITA/mcu.kicad_sch (KiCad schematic)
At the start: 60 parts, among them J1 Conn_02x10_Odd_Even, J2 Conn_02x06_Odd_Even, J3 Conn_02x13_Odd_Even, J4 15910060, SW1 SKRPABE010, SW2 SKRPABE010, SW3 SKRPABE010, U1 MX25UW25645GXDI00, U2 STM32H7S3Z8Tx, X1 24MHz

Commit message: Modified wiring between ICs.
Connections:
- net FDCAN2_RX: now also J1.10 (Pin_10); no longer J1.14 (Pin_14)
- net FDCAN2_TX: now also J1.12 (Pin_12); no longer J1.16 (Pin_16)
- net GND: now also J1.18 (Pin_18), J1.20 (Pin_20)
- net I2C2_SCL: now also J1.14 (Pin_14); no longer J1.18 (Pin_18)
- net I2C2_SDA: now also J1.16 (Pin_16); no longer J1.20 (Pin_20)
- net OSPI_CS: now reaches R2.1, U1.C2 (CS), U2.64 (PO0)
- net OSPI_SIO4: now reaches U1.D5 (SIO4), U2.47 (PP4)
- net OSPI_SIO2: now reaches U1.C4 (SIO2), U2.48 (PP2)
- net OSPI_SIO3: now reaches U1.D4 (SIO3), U2.49 (PP3)
- net OSPI_SCLK: now reaches U1.B2 (SCLK), U2.53 (PO4)
- net OSPI_SIO5: now reaches U1.E3 (SIO5), U2.54 (PP5)
- net OSPI_SIO0: now reaches U1.D3 (SIO0), U2.55 (PP0)
- net OSPI_SIO6: now reaches U1.E2 (SIO6), U2.58 (PP6)
- net OSPI_DQS: now reaches U1.C3 (DQS), U2.59 (PO2)
- net OSPI_SIO7: now reaches U1.E1 (SIO7), U2.60 (PP7)
- net OSPI_SIO1: now reaches U1.D2 (SIO1), U2.61 (PP1)
- net SAI2A_SCK: now reaches U2.72 (PD13)
- net SAI_DATA_IN renamed SAI1B_DATA_OUT
- net SAI_DATA_OUT renamed SAI1A_DATA_IN
- net SAI_FS renamed SAI1A_FS
- net SAI_SCK renamed SAI1A_SCK
- net USART3_CTS renamed SAI2A_DATA_OUT
- net SAI2A_DATA_OUT: no longer J1.10 (Pin_10)
- net USART3_RTS renamed SAI2A_FS
- net SAI2A_FS: no longer J1.12 (Pin_12)
- no-connect marks 14 -> 13

Commit message: Added some resistors and Schottky diode.
Parts:
- added D6: D_Schottky, Diode_SMD:D_SOD-523, symbol Device:D_Schottky
- renumbered J2 to J1, J1 to J2
Connections:
- net NRST: now also D6.1 (K); no longer U1.A4 (RESET)
- new net: D6.2 (A), U1.A4 (RESET)

Commit message: Improved some routes.
Connections:
- net SAI1B_DATA_OUT: no longer names the net of U2.9 (PE3)
- no-connect marks 13 -> 14

Commit message: Fixed some mistakes.
switched 5V and 5V_UCPD.
switched VREFP and VREFM.
Parts:
- removed C7: 100nF, Capacitor_SMD:C_0201_0603Metric, symbol Device:C
Connections:
- net 3V3: now also U2.24 (VREFP); no longer U2.23 (VREFM)
- net GND: now also U2.23 (VREFM); no longer U2.24 (VREFP)
Other:
- moved on the sheet: C10, C11, C12, C13, C14, C15, C16, C17, C18, C22, C23, C8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

Commit message: Changed pin assignments for J4 and J6.
Parts:
- J1: footprint Connector_PinHeader_2.54mm:PinHeader_2x06_P2.54mm_Vertical -> Connector_PinSocket_2.54mm:PinSocket_2x06_P2.54mm_Vertical
- J2: footprint Connector_PinHeader_2.54mm:PinHeader_2x10_P2.54mm_Vertical -> Connector_PinSocket_2.54mm:PinSocket_2x10_P2.54mm_Vertical
- J3: footprint Connector_PinHeader_2.54mm:PinHeader_2x13_P2.54mm_Vertical -> Connector_PinSocket_2.54mm:PinSocket_2x13_P2.54mm_Vertical
Connections:
- net 3V3: now also J4.1 (Pin_1); no longer J4.5 (Pin_5)
- net ADC1_IN0: now also J1.4 (Pin_4); no longer J1.3 (Pin_3)
- net ADC1_IN10: now also J1.5 (Pin_5); no longer J1.6 (Pin_6)
- net ADC1_IN12: now also J1.8 (Pin_8); no longer J1.7 (Pin_7)
- net ADC1_IN13: now also J1.7 (Pin_7); no longer J1.8 (Pin_8)
- net ADC1_IN15: now also J1.10 (Pin_10); no longer J1.9 (Pin_9)
- net ADC1_IN3: now also J1.3 (Pin_3); no longer J1.4 (Pin_4)
- net ADC1_IN5: now also J1.6 (Pin_6); no longer J1.5 (Pin_5)
- net DEBUG_SWDIO: now also J4.2 (Pin_2); no longer J4.6 (Pin_6)
- net ETH_MDC: now also J3.14 (Pin_14); no longer J3.13 (Pin_13)
- net ETH_MDIO: now also J3.6 (Pin_6); no longer J3.5 (Pin_5)
- net ETH_MII_RX_ER: now also J3.24 (Pin_24); no longer J3.23 (Pin_23)
- net ETH_RMII_CRS_DV: now also J3.8 (Pin_8); no longer J3.7 (Pin_7)
- net ETH_RMII_INTN: now also J3.20 (Pin_20); no longer J3.19 (Pin_19)
- net ETH_RMII_REF_CLK: now also J3.4 (Pin_4); no longer J3.3 (Pin_3)
- net ETH_RMII_RXD0: now also J3.16 (Pin_16); no longer J3.15 (Pin_15)
- net ETH_RMII_RXD1: now also J3.18 (Pin_18); no longer J3.17 (Pin_17)
- net ETH_RMII_TXD0: now also J3.10 (Pin_10); no longer J3.9 (Pin_9)
- net ETH_RMII_TXD1: now also J3.12 (Pin_12); no longer J3.11 (Pin_11)
- net ETH_RMII_TX_EN: now also J3.22 (Pin_22); no longer J3.21 (Pin_21)
- net FDCAN2_RX: now also J2.9 (Pin_9); no longer J2.10 (Pin_10)
- net FDCAN2_TX: now also J2.11 (Pin_11); no longer J2.12 (Pin_12)
- net GND: now also J1.9 (Pin_9), J2.17 (Pin_17), J3.23 (Pin_23), J4.5 (Pin_5); no longer J1.10 (Pin_10), J2.18 (Pin_18), J3.24 (Pin_24), J4.1 (Pin_1)
- net I2C2_SCL: now also J2.13 (Pin_13); no longer J2.14 (Pin_14)
- net I2C2_SDA: now also J2.15 (Pin_15); no longer J2.16 (Pin_16)
- net I2S3_CK: now also J2.12 (Pin_12); no longer J2.11 (Pin_11)
- net I2S3_SDI: now also J2.18 (Pin_18); no longer J2.17 (Pin_17)
- net I2S3_SDO: now also J2.16 (Pin_16); no longer J2.15 (Pin_15)
- net I2S3_WS: now also J2.14 (Pin_14); no longer J2.13 (Pin_13)
- net LPUART1_CTS: now also J2.8 (Pin_8); no longer J2.7 (Pin_7)
- net LPUART1_RTS: now also J2.10 (Pin_10); no longer J2.9 (Pin_9)
- net LPUART1_RX: now also J2.6 (Pin_6); no longer J2.5 (Pin_5)
- net LPUART1_TX: now also J2.4 (Pin_4); no longer J2.3 (Pin_3)
- net NRST: now also J4.6 (Pin_6); no longer J4.2 (Pin_2)
- net SDMMC2_CK: now also J3.3 (Pin_3); no longer J3.4 (Pin_4)
- net SDMMC2_CMD: now also J3.5 (Pin_5); no longer J3.6 (Pin_6)
- net SDMMC2_D0: now also J3.7 (Pin_7); no longer J3.8 (Pin_8)
- net SDMMC2_D1: now also J3.9 (Pin_9); no longer J3.10 (Pin_10)
- net SDMMC2_D2: now also J3.11 (Pin_11); no longer J3.12 (Pin_12)
- net SDMMC2_D3: now also J3.13 (Pin_13); no longer J3.14 (Pin_14)
- net SDMMC2_D4: now also J3.15 (Pin_15); no longer J3.16 (Pin_16)
- net SDMMC2_D5: now also J3.17 (Pin_17); no longer J3.18 (Pin_18)
- net SDMMC2_D6: now also J3.19 (Pin_19); no longer J3.20 (Pin_20)
- net SDMMC2_D7: now also J3.21 (Pin_21); no longer J3.22 (Pin_22)
- net USART3_CK: now also J2.7 (Pin_7); no longer J2.8 (Pin_8)
- net USART3_RX: now also J2.5 (Pin_5); no longer J2.6 (Pin_6)
- net USART3_TX: now also J2.3 (Pin_3); no longer J2.4 (Pin_4)
