File: KiCad/OTO_NO_ITA/OTO_NO_ITA.kicad_pcb (KiCad board)
At the start: 4 copper layers, 73 x 72 mm, 121 parts, among them J1 Conn_02x10_Odd_Even, J2 Conn_02x06_Odd_Even, J3 Conn_02x13_Odd_Even, J4 15910060, J5 Conn_02x07_Odd_Even, J6 15910060, J7 Conn_01x02, J8 Conn_01x02, J9 UB1611-HGN, Q1 STD2805T4, Q2 STL40DN3LLH5, Q3 STL40DN3LLH5, SW1 SKRPABE010, SW2 SKRPABE010, SW3 SKRPABE010, SW4 SKRPABE010, U1 MX25UW25645GXDI00, U2 STM32H7S3Z8Tx, U3 ADAU1466WBCPZ300RL, U4 ADM811TARTZ, U5 AP7361EA-33E-13, U6 AP2127N-1.8TRG1, U7 TCPP03-M20, U8 ESDA25P35-1U1M, U9 ECMF2-40A100N6, X1 24MHz, X2 12.288MHz

Commit message: Changed layer from 4 to 6.
Routing:
- added copper zone on In4.Cu, net 1V8
- added copper zone on In4.Cu, net 3V3
- added copper zone on In4.Cu, net DVDD
- added copper zone on In3.Cu, net GND
- removed copper zone on In2.Cu, net 1V8
- removed copper zone on In2.Cu, net 3V3
- removed copper zone on In2.Cu, net DVDD
Other:
- copper layers 4 -> 6

Commit message: Improved board design.
Connections:
- net Net-(U1-CS) renamed /MCU/OSPI_CS
- net Net-(U1-DQS) renamed /MCU/OSPI_DQS
- net Net-(U1-SCLK) renamed /MCU/OSPI_SCLK
- net Net-(U1-SIO0) renamed /MCU/OSPI_SIO0
- net Net-(U1-SIO1) renamed /MCU/OSPI_SIO1
- net Net-(U1-SIO2) renamed /MCU/OSPI_SIO2
- net Net-(U1-SIO3) renamed /MCU/OSPI_SIO3
- net Net-(U1-SIO4) renamed /MCU/OSPI_SIO4
- net Net-(U1-SIO5) renamed /MCU/OSPI_SIO5
- net Net-(U1-SIO6) renamed /MCU/OSPI_SIO6
- net Net-(U1-SIO7) renamed /MCU/OSPI_SIO7
- J1 pad 10: /MCU/USART3_CTS -> /MCU/FDCAN2_RX
- J1 pad 12: /MCU/USART3_RTS -> /MCU/FDCAN2_TX
- J1 pad 14: /MCU/FDCAN2_RX -> /MCU/I2C2_SCL
- J1 pad 16: /MCU/FDCAN2_TX -> /MCU/I2C2_SDA
- J1 pad 18: /MCU/I2C2_SCL -> GND
- J1 pad 20: /MCU/I2C2_SDA -> GND
- U2 pad 12: /DSP/DSP_SDATA_IN0 -> /DSP/DSP_SDATA_OUT0
- U2 pad 68: /MCU/USART3_CTS -> /DSP/DSP_SDATA_IN0
- U2 pad 71: /MCU/USART3_RTS -> /DSP/DSP_LRCLK_IN0
- U2 pad 72: unconnected-(U2-PD13-Pad72) -> /DSP/DSP_BCLK_IN0
- U2 pad 9: /DSP/DSP_SDATA_OUT0 -> /MCU/SAI1B_DATA_OUT
Routing:
- net /DSP/DSP_BCLK_IN0: track 0.00 -> 45.3 mm, vias 0 -> 2
- net /DSP/DSP_LRCLK_IN0: track 0.00 -> 44.0 mm, vias 0 -> 2
- net /MCU/USART3_CTS: track 24.9 -> 0.00 mm, vias 1 -> 0
- net /DSP/DSP_SDATA_IN0: track 21.6 -> 45.5 mm
- net /MCU/USART3_RTS: track 21.8 -> 0.00 mm, vias 1 -> 0
- net /MCU/SDMMC2_D5: track 45.4 -> 30.7 mm
- net /MCU/SDMMC2_D1: track 68.7 -> 58.3 mm
- net /MCU/SDMMC2_D4: track 42.1 -> 32.5 mm, vias 0 -> 1
- net /MCU/SDMMC2_D6: track 67.2 -> 57.6 mm
- net /DSP/DSP_SDATA_OUT0: track 18.7 -> 27.9 mm
- net /MCU/SDMMC2_D0: track 65.6 -> 57.2 mm
- net GND: track 149.3 -> 141.3 mm
- net /MCU/I2C2_SCL: track 55.1 -> 62.9 mm
- net VBUS: track 9.12 -> 2.36 mm
- net /MCU/SDMMC2_D3: track 46.4 -> 40.8 mm, vias 0 -> 1
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- added copper zone on In3.Cu, net 1V8
- added copper zone on In3.Cu, net 3V3
- added copper zone on In3.Cu, net 5V
- added copper zone on In3.Cu, net 5V_UCPD
- added copper zone on F.Cu, net DVDD
- added copper zone on In4.Cu, net GND
- added copper zone on In3.Cu, net VBUS
- removed copper zone on In4.Cu, net 1V8
- removed copper zone on In4.Cu, net 3V3
- removed copper zone on B.Cu, net 5V
- removed copper zone on B.Cu, net 5V_UCPD
- removed copper zone on In4.Cu, net DVDD
- removed copper zone on In3.Cu, net GND

Commit message: Improved GND plane.
Routing:
- net GND: track 141.3 -> 142.9 mm, vias 125 -> 121
- net /MCU/I2S3_SDO: track 46.5 -> 45.1 mm
- net /MCU/DEBUG_SWDIO: track 32.1 -> 31.0 mm
- net /MCU/I2S3_WS: track 28.5 -> 29.2 mm

Commit message: Modified the date.
Other:
- board text added: "2025/04/23"
- board text removed: "2025/04/21"
Changed lines of the file:
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@@
 		)
 	)
-	(gr_text "2025/04/21"
+	(gr_text "2025/04/23"
 		(at 148.367143 96.42 0)
 		(layer "F.SilkS")
