File: KiCad/OTO_NO_ITA/OTO_NO_ITA.kicad_pcb (KiCad board)
At the start: 6 copper layers, 73 x 72 mm, 132 parts, among them J1 Conn_02x06_Odd_Even, J2 Conn_02x10_Odd_Even, J3 Conn_02x13_Odd_Even, J4 15910060, J5 Conn_02x07_Odd_Even, J6 Conn_02x04_Odd_Even, J7 Conn_01x02, J8 Conn_01x02, J9 UB1611-HGN, Q1 STD2805T4, Q2 STL40DN3LLH5, Q3 STL40DN3LLH5, SW1 SKRPABE010, SW2 SKRPABE010, SW3 SKRPABE010, SW4 SKRPABE010, U1 MX25UW25645GXDI00, U2 STM32H7S3Z8Tx, U3 ADAU1466WBCPZ300RL, U4 ADM811TARTZ, U5 AP7361EA-33E-13, U6 AP2127N-1.8TRG1, U7 TCPP03-M20, U8 ESDA25P35-1U1M, U9 ECMF2-40A100N6, X1 24MHz, X2 12.288MHz

Commit message: Change J7 and J8(5V in/out connector) to JST PH.
Parts:
- J7, J8: footprint Connector_PinHeader_2.54mm:PinHeader_1x02_P2.54mm_Vertical -> Connector_JST:JST_PH_S2B-PH-K_1x02_P2.00mm_Horizontal
- moved J8 3.48 mm to (103.2, 122.3), turned to -90 degrees
- moved J7 3.03 mm to (109.8, 130.2), turned to 0 degrees
- moved D5 2.88 mm to (109.8, 125.8)
Routing:
- net Net-(D5-A): track 0.00 -> 2.90 mm
- removed copper zone on F.Cu, net Net-(D5-A)
Other:
- board text added: "2025/05/02"
- board text removed: "2025/04/30"

Commit message: Improved some routes.
Connections:
- U2 pad 9: /MCU/SAI1B_DATA_OUT -> unconnected-(U2-PE3-Pad9)
Routing:
- net /MCU/SDMMC2_D2: track 62.3 -> 53.4 mm
- net /MCU/SDMMC2_CMD: track 65.2 -> 58.1 mm
- net /MCU/SDMMC2_CK: track 66.1 -> 59.9 mm
- net /DSP/DSP_LRCLK_OUT0: track 24.5 -> 18.9 mm
- net /DSP/DSP_BCLK_OUT0: track 25.1 -> 19.6 mm
- net /DSP/DSP_SDATA_OUT0: track 25.4 -> 20.5 mm
- net /DSP/DSP_LRCLK_IN0: track 39.9 -> 36.2 mm
- net /DSP/DSP_BCLK_IN0: track 42.3 -> 38.6 mm
- net /DSP/DSP_SDATA_IN0: track 39.9 -> 36.3 mm
- net /MCU/NRST: track 92.3 -> 89.3 mm, vias 3 -> 2
- net /DSP/CLKOUT: track 61.5 -> 58.9 mm
- net /MCU/SDMMC2_D3: track 40.8 -> 43.1 mm
- net /MCU/ETH_RMII_INTN: track 53.5 -> 52.0 mm
- net /MCU/UCPD_ISENSE: track 47.6 -> 46.5 mm
- net /MCU/I2S3_SDO: track 45.1 -> 44.2 mm
Other:
- board text added: "2025/05/09"
- board text removed: "2025/05/02"

Commit message: Fixed some JLCPCB part No.
Parts:
- J4: value 15910060 -> (none)
Other:
- board text added: "2025/05/13"
- board text removed: "2025/05/09"
Changed lines of the file:
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@@
 			)
 		)
-		(property "LCSC" "C2858031"
+		(property "LCSC" "C162274"
 			(at 0 0 0)
 			(layer "F.SilkS")
@@
 			)
 		)
-		(property "LCSC" "C162273"
+		(property "LCSC" "C126632"
 			(at 0 0 0)
 			(layer "F.SilkS")
@@
 			)
 		)
-		(property "LCSC" "C2858031"
+		(property "LCSC" "C162274"
 			(at 0 0 0)
 			(layer "F.SilkS")
@@
 			)
 		)
-		(property "LCSC" "C361059"
+		(property "LCSC" "C77386"
 			(at 0 0 0)
 			(layer "F.SilkS")
@@
 			)
 		)
-		(property "Value" "15910060"
+		(property "Value" ""
 			(at 1.27 7.41 90)
 			(layer "F.Fab")
@@
 			)
 		)
-		(property "LCSC" "C2858031"
+		(property "LCSC" "C162274"
 			(at 0 0 0)
 			(layer "F.SilkS")
@@
 			)
 		)
-		(property "LCSC" "C361059"
+		(property "LCSC" "C77386"
 			(at 0 0 0)
 			(layer "F.SilkS")
@@
 			)
 		)
-		(property "LCSC" "C361059"
+		(property "LCSC" "C77386"
 			(at 0 0 0)
 			(layer "F.SilkS")
@@
 		(layer "F.SilkS")
 	)
+	(gr_circle
+		(center 121.475 126.775)
+		(end 121.475 126.675)
+		(stroke
+			(width 0.15)
+			(type default)
+		)
+		(fill no)
+		(layer "F.SilkS")
+	)
 	(gr_line
 		(start 115.25 99.9)
@@
 		)
 	)
-	(gr_text "2025/05/09"
+	(gr_text "2025/05/13"
 		(at 148.367143 96.42 0)
 		(layer "F.SilkS")
@@
 		(name "$teardrop_padvia$")
 		(hatch full 0.1)
+		(priority 30001)
+		(attr
+			(teardrop
+				(type padvia)
+			)
+		)
+		(connect_pads yes
+			(clearance 0)
+		)
+		(min_thickness 0.0254)
+		(filled_areas_thickness no)
+		(fill yes
+			(thermal_gap 0.5)
+			(thermal_bridge_width 0.5)
+			(island_removal_mode 1)
+			(island_area_min 10)
+		)
+		(polygon
+			(pts
+				(xy 112.347151 72.799994) (xy 112.629994 72.517151) (xy 112.923667 71.305827) (xy 112.089293 71.139293)
+				(xy 111.383251 71.612235)
+			)
+		)
+	)
+	(zone
+		(net 2)
+		(net_name "GND")
+		(layer "F.Cu")
+		(name "$teardrop_padvia$")
+		(hatch full 0.1)
 		(priority 30055)
 		(attr
@@
 	)
 	(zone
+		(net 5)
+		(net_name "3V3")
+		(layer "F.Cu")
+		(name "$teardrop_padvia$")
+		(hatch full 0.1)
+		(priority 30000)
+		(attr
+			(teardrop
+				(type padvia)
+			)
+		)
+		(connect_pads yes
+			(clearance 0)
+		)
+		(min_thickness 0.0254)
+		(filled_areas_thickness no)
+		(fill yes
+			(thermal_gap 0.5)
+			(thermal_bridge_width 0.5)
+			(island_removal_mode 1)
+			(island_area_min 10)
+		)
+		(polygon
+			(pts
+				(xy 114.425 72.823667) (xy 114.825 72.823667) (xy 115.336749 71.612235) (xy 114.63 71.139) (xy 113.796333 71.305827)
+			)
+		)
+	)
+	(zone
 		(net 184)
 		(net_name "Net-(U3-SDATA_OUT0)")
@@
 	)
 	(zone
-		(net 2)
-		(net_name "GND")
-		(layer "F.Cu")
-		(name "$teardrop_padvia$")
-		(hatch full 0.1)
-		(priority 30002)
-		(attr
-			(teardrop
-				(type padvia)
-			)
-		)
-		(connect_pads yes
-			(clearance 0)
-		)
-		(min_thickness 0.0254)
-		(filled_areas_thickness no)
-		(fill yes
-			(thermal_gap 0.5)
-			(thermal_bridge_width 0.5)
-			(island_removal_mode 1)
-			(island_area_min 10)
-		)
-		(polygon
-			(pts
-				(xy 112.347151 72.799994) (xy 112.629994 72.517151) (xy 112.923667 71.305827) (xy 112.089293 71.139293)
-				(xy 111.383251 71.612235)
-			)
-		)
-	)
-	(zone
 		(net 148)
 		(net_name "/MCU/I2S3_CK")
@@
 	)
 	(zone
-		(net 5)
-		(net_name "3V3")
-		(layer "F.Cu")
-		(name "$teardrop_padvia$")
-		(hatch full 0.1)
-		(priority 30001)
-		(attr
-			(teardrop
-				(type padvia)
-			)
-		)
-		(connect_pads yes
-			(clearance 0)
-		)
-		(min_thickness 0.0254)
-		(filled_areas_thickness no)
-		(fill yes
-			(thermal_gap 0.5)
-			(thermal_bridge_width 0.5)
-			(island_removal_mode 1)
-			(island_area_min 10)
-		)
-		(polygon
-			(pts
-				(xy 114.425 72.823667) (xy 114.825 72.823667) (xy 115.336749 71.612235) (xy 114.63 71.139) (xy 113.796333 71.305827)
-			)
-		)
-	)
-	(zone
 		(net 138)
 		(net_name "/MCU/USART3_RX")
@@
 	)
 	(zone
+		(net 10)
+		(net_name "/MCU/NRST")
+		(layer "F.Cu")
+		(name "$teardrop_padvia$")
+		(hatch full 0.1)
+		(priority 30002)
+		(attr
+			(teardrop
+				(type padvia)
+			)
+		)
+		(connect_pads yes
+			(clearance 0)
+		)
+		(min_thickness 0.0254)
+		(filled_areas_thickness no)
+		(fill yes
+			(thermal_gap 0.5)
+			(thermal_bridge_width 0.5)
+			(island_removal_mode 1)
+			(island_area_min 10)
+		)
+		(polygon
+			(pts
+				(xy 110.652144 69.878921) (xy 110.828921 69.702144) (xy 110.383667 68.434173) (xy 109.549293 68.599293)
+				(xy 109.384173 69.433667)
+			)
+		)
+	)
+	(zone
 		(net 2)
 		(net_name "GND")
@@
 	)
 	(zone
-		(net 10)
-		(net_name "/MCU/NRST")
-		(layer "F.Cu")
-		(name "$teardrop_padvia$")
-		(hatch full 0.1)
-		(priority 30005)
-		(attr
-			(teardrop
-				(type padvia)
-			)
-		)
-		(connect_pads yes
-			(clearance 0)
-		)
-		(min_thickness 0.0254)
-		(filled_areas_thickness no)
-		(fill yes
-			(thermal_gap 0.5)
-			(thermal_bridge_width 0.5)
-			(island_removal_mode 1)
-			(island_area_min 10)
-		)
-		(polygon
-			(pts
-				(xy 110.652144 69.878921) (xy 110.828921 69.702144) (xy 110.383667 68.434173) (xy 109.549293 68.599293)
-				(xy 109.384173 69.433667)
-			)
-		)
-	)
-	(zone
 		(net 61)
 		(net_name "Net-(U7-C_BIAS)")
@@
 	)
 	(zone
-		(net 31)
-		(net_name "/MCU/DEBUG_SWCLK")
-		(layer "B.Cu")
-		(name "$teardrop_padvia$")
-		(hatch full 0.1)
-		(priority 30012)
-		(attr
-			(teardrop
-				(type padvia)
-			)
-		)
-		(connect_pads yes
-			(clearance 0)
-		)
-		(min_thickness 0.0254)
-		(filled_areas_thickness no)
-		(fill yes
-			(thermal_gap 0.5)
-			(thermal_bridge_width 0.5)
-			(island_removal_mode 1)
-			(island_area_min 10)
-		)
-		(polygon
-			(pts
-				(xy 113.068 69.82679) (xy 113.318 69.82679) (xy 112.923667 68.434173) (xy 112.09 68.599) (xy 111.924173 69.433667)
-			)
-		)
-	)
-	(zone
 		(net 3)
 		(net_name "/USB/CC2")
@@
 	)
 	(zone
+		(net 30)
+		(net_name "/MCU/DEBUG_SWDIO")
+		(layer "B.Cu")
+		(name "$teardrop_padvia$")
+		(hatch full 0.1)
+		(priority 30000)
+		(attr
+			(teardrop
+				(type padvia)
+			)
+		)
+		(connect_pads yes
+			(clearance 0)
+		)
+		(min_thickness 0.0254)
+		(filled_areas_thickness no)
+		(fill yes
+			(thermal_gap 0.5)
+			(thermal_bridge_width 0.5)
+			(island_removal_mode 1)
+			(island_area_min 10)
+		)
+		(polygon
+			(pts
+				(xy 115.732144 69.878921) (xy 115.908921 69.702144) (xy 115.463667 68.434173) (xy 114.629293 68.599293)
+				(xy 114.464173 69.433667)
+			)
+		)
+	)
+	(zone
 		(net 9)
 		(net_name "/DSP/DSP_RESET")
@@
 	)
 	(zone
-		(net 125)
-		(net_name "/MCU/ETH_RMII_INTN")
+		(net 31)
+		(net_name "/MCU/DEBUG_SWCLK")
 		(layer "B.Cu")
 		(name "$teardrop_padvia$")
 		(hatch full 0.1)
-		(priority 30002)
+		(priority 30001)
 		(attr
 			(teardrop
@@
 		(polygon
 			(pts
-				(xy 161.586333 98.98) (xy 161.586333 99.18) (xy 162.797765 99.786749) (xy 163.271 99.08) (xy 162.797765 98.373251)
+				(xy 113.068 69.82679) (xy 113.318 69.82679) (xy 112.923667 68.434173) (xy 112.09 68.599) (xy 111.924173 69.433667)
 			)
 		)
 	)
 	(zone
-		(net 150)
-		(net_name "/MCU/LPUART1_RX")
+		(net 125)
+		(net_name "/MCU/ETH_RMII_INTN")
 		(layer "B.Cu")
 		(name "$teardrop_padvia$")
 		(hatch full 0.1)
-		(priority 30006)
+		(priority 30002)
 		(attr
 			(teardrop
@@
 		(polygon
 			(pts
-				(xy 100.889822 80.021243) (xy 101.031243 79.879822) (xy 100.603667 78.594173) (xy 99.769293 78.759293)
-				(xy 99.604173 79.593667)
+				(xy 161.586333 98.98) (xy 161.586333 99.18) (xy 162.797765 99.786749) (xy 163.271 99.08) (xy 162.797765 98.373251)
 			)
 		)
 	)
 	(zone
-		(net 143)
-		(net_name "/MCU/I2S3_WS")
+		(net 150)
+		(net_name "/MCU/LPUART1_RX")
 		(layer "B.Cu")
 		(name "$teardrop_padvia$")
 		(hatch full 0.1)
-		(priority 30086)
+		(priority 30006)
 		(attr
 			(teardrop
@@
 		(polygon
 			(pts
-				(xy 118.023917 99.010657) (xy 118.165338 99.152078) (xy 118.574441 98.741671) (xy 118.325707 98.574293)
-				(xy 118.030764 98.516473)
+				(xy 100.889822 80.021243) (xy 101.031243 79.879822) (xy 100.603667 78.594173) (xy 99.769293 78.759293)
+				(xy 99.604173 79.593667)
 			)
 		)
 	)
 	(zone
-		(net 30)
-		(net_name "/MCU/DEBUG_SWDIO")
+		(net 143)
+		(net_name "/MCU/I2S3_WS")
 		(layer "B.Cu")
 		(name "$teardrop_padvia$")
 		(hatch full 0.1)
-		(priority 30000)
+		(priority 30086)
 		(attr
 			(teardrop
@@
 		(polygon
 			(pts
-				(xy 115.732144 69.878921) (xy 115.908921 69.702144) (xy 115.463667 68.434173) (xy 114.629293 68.599293)
-				(xy 114.464173 69.433667)
+				(xy 118.023917 99.010657) (xy 118.165338 99.152078) (xy 118.574441 98.741671) (xy 118.325707 98.574293)
+				(xy 118.030764 98.516473)
 			)
 		)
