File: KiCad/OTO_NO_ITA/OTO_NO_ITA.kicad_pcb (KiCad board)
At the start: 6 copper layers, 73 x 72 mm, 132 parts, among them J1 Conn_02x06_Odd_Even, J2 Conn_02x10_Odd_Even, J3 Conn_02x13_Odd_Even, J5 Conn_02x07_Odd_Even, J6 Conn_02x04_Odd_Even, J7 Conn_01x02, J8 Conn_01x02, J9 UB1611-HGN, Q1 STD2805T4, Q2 STL40DN3LLH5, Q3 STL40DN3LLH5, SW1 SKRPABE010, SW2 SKRPABE010, SW3 SKRPABE010, SW4 SKRPABE010, U1 MX25UW25645GXDI00, U2 STM32H7S3Z8Tx, U3 ADAU1466WBCPZ300RL, U4 ADM811TARTZ, U5 AP7361EA-33E-13, U6 AP2127N-1.8TRG1, U7 TCPP03-M20, U8 ESDA25P35-1U1M, U9 ECMF2-40A100N6, X1 24MHz, X2 12.288MHz

Commit message: Fixed U2 footprint.
Parts:
- moved C4 1.25 mm to (132.0, 74.3)
- moved C3 1.25 mm to (133.2, 74.4)
- moved R3 1.25 mm to (132.1, 76.1)
- moved C21 1.10 mm to (125.7, 69.7)
- moved R2 1.10 mm to (127.6, 69.7)
- moved C20 1.10 mm to (125.7, 68.3)
- moved C25 0.90 mm to (120.6, 75.8)
- moved C24 0.90 mm to (119.5, 75.8)
Routing:
- net 1V8: track 29.6 -> 31.5 mm
- net GND: track 144.3 -> 146.1 mm
- net /MCU/OSPI_CS: track 22.4 -> 21.3 mm
- net Net-(U1-ECS): track 3.01 -> 3.90 mm
Other:
- board text added: "2025/05/14"
- board text removed: "2025/05/13"

Commit message: Fixed some mistakes.
switched 5V and 5V_UCPD.
switched VREFP and VREFM.
Parts:
- removed C7: 100nF, Capacitor_SMD:C_0201_0603Metric
- J4: value (none) -> 15910060
- moved C22 1.00 mm to (140.1, 92.3)
- moved C23 1.00 mm to (139.8, 91.4)
Connections:
- C62 pad 1: 5V -> 5V_UCPD
- C65 pad 1: 5V -> 5V_UCPD
- D5 pad 1: 5V_UCPD -> 5V
- J8 pad 1: 5V -> 5V_UCPD
- U2 pad 23: 3V3 -> GND
- U2 pad 24: GND -> 3V3
- U5 pad 1: 5V -> 5V_UCPD
- U6 pad 3: 5V -> 5V_UCPD
Routing:
- net 5V_UCPD: track 0.00 -> 6.06 mm, vias 6 -> 4
- net GND: track 146.1 -> 146.7 mm, vias 122 -> 120
- net 3V3: track 82.3 -> 81.8 mm, vias 33 -> 32
- net 5V: vias 3 -> 6
Other:
- board text added: "2025/05/23"
- board text added: "rev.B"
- board text removed: "2025/05/14"
- board text removed: "rev.A"

Commit message: Changed pin assignments for J4 and J6.
Parts:
- J1: footprint Connector_PinHeader_2.54mm:PinHeader_2x06_P2.54mm_Vertical -> Connector_PinSocket_2.54mm:PinSocket_2x06_P2.54mm_Vertical
- J2: footprint Connector_PinHeader_2.54mm:PinHeader_2x10_P2.54mm_Vertical -> Connector_PinSocket_2.54mm:PinSocket_2x10_P2.54mm_Vertical
- J3: footprint Connector_PinHeader_2.54mm:PinHeader_2x13_P2.54mm_Vertical -> Connector_PinSocket_2.54mm:PinSocket_2x13_P2.54mm_Vertical
- J5: footprint Connector_PinHeader_2.54mm:PinHeader_2x07_P2.54mm_Vertical -> Connector_PinSocket_2.54mm:PinSocket_2x07_P2.54mm_Vertical
- moved J6 8.03 mm to (153.1, 129.6), turned to -90 degrees
- moved C34 4.46 mm to (109.8, 73.6), turned to 180 degrees
- moved J1 2.54 mm to (137.9, 68.6)
- moved J2 2.54 mm to (102.3, 73.7)
- moved J3 2.54 mm to (165.8, 76.2)
- moved J5 2.54 mm to (165.8, 111.8)
Connections:
- J1 pad 10: GND -> /MCU/ADC1_IN15
- J1 pad 3: /MCU/ADC1_IN0 -> /MCU/ADC1_IN3
- J1 pad 4: /MCU/ADC1_IN3 -> /MCU/ADC1_IN0
- J1 pad 5: /MCU/ADC1_IN5 -> /MCU/ADC1_IN10
- J1 pad 6: /MCU/ADC1_IN10 -> /MCU/ADC1_IN5
- J1 pad 7: /MCU/ADC1_IN12 -> /MCU/ADC1_IN13
- J1 pad 8: /MCU/ADC1_IN13 -> /MCU/ADC1_IN12
- J1 pad 9: /MCU/ADC1_IN15 -> GND
- J2 pad 10: /MCU/FDCAN2_RX -> /MCU/LPUART1_RTS
- J2 pad 11: /MCU/I2S3_CK -> /MCU/FDCAN2_TX
- J2 pad 12: /MCU/FDCAN2_TX -> /MCU/I2S3_CK
- J2 pad 13: /MCU/I2S3_WS -> /MCU/I2C2_SCL
- J2 pad 14: /MCU/I2C2_SCL -> /MCU/I2S3_WS
- J2 pad 15: /MCU/I2S3_SDO -> /MCU/I2C2_SDA
- J2 pad 16: /MCU/I2C2_SDA -> /MCU/I2S3_SDO
- J2 pad 17: /MCU/I2S3_SDI -> GND
- J2 pad 18: GND -> /MCU/I2S3_SDI
- J2 pad 3: /MCU/LPUART1_TX -> /MCU/USART3_TX
- J2 pad 4: /MCU/USART3_TX -> /MCU/LPUART1_TX
- J2 pad 5: /MCU/LPUART1_RX -> /MCU/USART3_RX
- J2 pad 6: /MCU/USART3_RX -> /MCU/LPUART1_RX
- J2 pad 7: /MCU/LPUART1_CTS -> /MCU/USART3_CK
- J2 pad 8: /MCU/USART3_CK -> /MCU/LPUART1_CTS
- J2 pad 9: /MCU/LPUART1_RTS -> /MCU/FDCAN2_RX
- J3 pad 10: /MCU/SDMMC2_D1 -> /MCU/ETH_RMII_TXD0
- J3 pad 11: /MCU/ETH_RMII_TXD1 -> /MCU/SDMMC2_D2
- J3 pad 12: /MCU/SDMMC2_D2 -> /MCU/ETH_RMII_TXD1
- J3 pad 13: /MCU/ETH_MDC -> /MCU/SDMMC2_D3
- J3 pad 14: /MCU/SDMMC2_D3 -> /MCU/ETH_MDC
- J3 pad 15: /MCU/ETH_RMII_RXD0 -> /MCU/SDMMC2_D4
- J3 pad 16: /MCU/SDMMC2_D4 -> /MCU/ETH_RMII_RXD0
- J3 pad 17: /MCU/ETH_RMII_RXD1 -> /MCU/SDMMC2_D5
- J3 pad 18: /MCU/SDMMC2_D5 -> /MCU/ETH_RMII_RXD1
- J3 pad 19: /MCU/ETH_RMII_INTN -> /MCU/SDMMC2_D6
- J3 pad 20: /MCU/SDMMC2_D6 -> /MCU/ETH_RMII_INTN
- J3 pad 21: /MCU/ETH_RMII_TX_EN -> /MCU/SDMMC2_D7
- J3 pad 22: /MCU/SDMMC2_D7 -> /MCU/ETH_RMII_TX_EN
- J3 pad 23: /MCU/ETH_MII_RX_ER -> GND
- J3 pad 24: GND -> /MCU/ETH_MII_RX_ER
- J3 pad 3: /MCU/ETH_RMII_REF_CLK -> /MCU/SDMMC2_CK
- J3 pad 4: /MCU/SDMMC2_CK -> /MCU/ETH_RMII_REF_CLK
- J3 pad 5: /MCU/ETH_MDIO -> /MCU/SDMMC2_CMD
- J3 pad 6: /MCU/SDMMC2_CMD -> /MCU/ETH_MDIO
- J3 pad 7: /MCU/ETH_RMII_CRS_DV -> /MCU/SDMMC2_D0
- J3 pad 8: /MCU/SDMMC2_D0 -> /MCU/ETH_RMII_CRS_DV
- J3 pad 9: /MCU/ETH_RMII_TXD0 -> /MCU/SDMMC2_D1
- J4 pad 1: GND -> 3V3
- J4 pad 2: /MCU/NRST -> /MCU/DEBUG_SWDIO
- J4 pad 5: 3V3 -> GND
- J4 pad 6: /MCU/DEBUG_SWDIO -> /MCU/NRST
- J5 pad 10: /DSP/SDATA_OUT2 -> /DSP/SDATA_OUT1
- J5 pad 11: /DSP/SDATA_IN1 -> /DSP/SDATA_IN2
- J5 pad 12: /DSP/SDATA_IN2 -> /DSP/SDATA_IN1
- J5 pad 5: /DSP/BCLK_OUT1 -> /DSP/BCLK_OUT2
- J5 pad 6: /DSP/BCLK_OUT2 -> /DSP/BCLK_OUT1
- J5 pad 7: /DSP/LRCLK_OUT1 -> /DSP/LRCLK_OUT2
- J5 pad 8: /DSP/LRCLK_OUT2 -> /DSP/LRCLK_OUT1
- J5 pad 9: /DSP/SDATA_OUT1 -> /DSP/SDATA_OUT2
Routing:
- net /DSP/USBi_SS: track 64.8 -> 83.7 mm
- net Net-(J6-Pin_2): track 13.3 -> 2.72 mm
- net /DSP/USBi_MOSI: track 52.8 -> 57.6 mm
- net /DSP/USBi_MISO: track 54.8 -> 51.4 mm
- net /MCU/DEBUG_SWDIO: track 31.0 -> 33.1 mm
- net /MCU/NRST: track 89.3 -> 87.7 mm
- net /DSP/USBi_SCLK: track 58.3 -> 59.3 mm
- net /DSP/SDATA_OUT2: track 40.8 -> 41.4 mm
Other:
- board text added: "2025/07/02"
- board text added: "rev.C"
- board text removed: "2025/05/23"
- board text removed: "rev.B"
