File: KiCad/OTO_NO_ITA/dsp.kicad_sch (KiCad schematic)
At the start: 1 part, among them U2 ADAU1466WBCPZ300RL

Commit message: Updated schematics.
Parts:
- added C10, C12, C14, C15, C16, C17, C19, C20, C21, C22, C27, C38: 100nF, symbol Device:C
- added C11, C13, C18, C23: 10uF, symbol Device:C
- added C24: 150pF, symbol Device:C
- added C25: 5.6nF, symbol Device:C
- added C26: 100nF, Capacitor_SMD:C_0402_1005Metric, symbol Device:C
- added C28, C29, C30, C31: 10nF, symbol Device:C
- added Q3: STD2805T4, symbol Transistor_BJT:Q_PNP_BCE
- added R5: 1k, symbol Device:R
- added R6: 4.32k, symbol Device:R
- added R7: 10k, symbol Device:R
- added R8: 33R, Resistor_SMD:R_0402_1005Metric, symbol Device:R
- added R9: 100k, symbol Device:R
- added SW1: SW_MEC_5G, symbol My_Parts:SW_MEC_5G
- added U8: ADM811TARTZ, symbol My_Parts:ADM811
- added X1: 12.288MHz, symbol Oscillator:SG-8002CE
Connections:
- net GND: now reaches U2.1 (DGND)
- net GND: now also U2.14 (PGND), U2.17 (DGND), U2.19 (DGND), U2.25 (DGND), U2.36 (DGND), U2.37 (DGND), U2.54 (DGND), U2.55 (DGND), U2.6 (AGND), U2.72 (DGND), U2.73 (EP(GND)), C10.2, C11.2, C12.2, C13.2, C14.2, C15.2, C16.2, C17.2, C18.2, C19.2, C20.2, C21.2, C22.2, C23.2, C26.1, C27.2, C28.2, C29.2, C30.2, C31.2, C38.2, R7.1, R9.1, SW1.3 (B), U8.1 (GND), X1.2 (GND)
- net 3V3: now reaches U2.15 (PVDD)
- net 3V3: now also U2.18 (IOVDD), U2.2 (IOVDD), U2.38 (IOVDD), U2.56 (IOVDD), U2.7 (AVDD), C10.1, C11.1, C12.1, C13.1, C19.1, C20.1, C21.1, C22.1, C23.1, C24.1, C25.2, C26.2, C27.1, Q3.3 (E), R5.1, U8.4 (VCC), X1.4 (Vcc)
- net at U2.16 (PLLFILT): now also C24.2, R6.2
- net DVDD: now reaches U2.20 (DVDD)
- net DVDD: now also U2.35 (DVDD), U2.53 (DVDD), U2.71 (DVDD), C14.1, C15.1, C16.1, C17.1, C18.1, C28.1, C29.1, C30.1, C31.1, Q3.2 (C)
- net MCLK: now reaches U2.21 (XTALIN/MCLK)
- net MCLK: now also R8.2
- net DSP_CLKOUT: now reaches U2.23 (CLKOUT)
- net ~{RESET}: now reaches U2.24 (RESET*)
- net ~{RESET}: now also R9.2, U8.2 (~{RESET})
- net at U2.3 (VDRIVE): now also Q3.1 (B), R5.2
- net DSP_MISO: now reaches U2.30 (MISO/SDA)
- net DSP_SCLK: now reaches U2.31 (SCLKC/SCL)
- net DSP_MOSI: now reaches U2.32 (MOSI/ADDR1)
- net DSP_SS: now reaches U2.33 (SS/ADDR0)
- net at U2.34 (SELFBOOT): now also R7.2
- net DSP_LRCLK_OUT0: now reaches U2.39 (LRCLK_OUT0/MP4)
- net DSP_BCLK_OUT0: now reaches U2.40 (BCLK_OUT0)
- net DSP_SDATA_OUT0: now reaches U2.41 (SDATA_OUT0)
- net DSP_BCLK_IN0: now reaches U2.57 (BCLK_IN0)
- net DSP_LRCLK_IN0: now reaches U2.58 (LRCLK_IN0/MP10)
- net DSP_SDATA_IN0: now reaches U2.59 (SDATA_IN0)
- new net: C25.1, R6.1
- new net: R8.1, X1.3 (OUT)
- new net DSP_RESET: C38.1, SW1.1 (A), U8.3 (~{MR})
- no-connect marks 0 -> 18
Other:
- note added: "to USBi"
- moved on the sheet: U2

Commit message: Updated schematics.
Parts:
- added J5, J6, J7: Conn_01x06, My_Parts:PinHeader_1x06_P2.54mm_Vertical, symbol Connector_Generic:Conn_01x06
Connections:
- net 3V3: now also J5.1 (Pin_1), J6.1 (Pin_1), J7.1 (Pin_1)
- net GND: now also J5.6 (Pin_6), J6.6 (Pin_6), J7.6 (Pin_6)
- net LRCLK_OUT1: now reaches U2.42 (LRCLK_OUT1/MP5)
- net LRCLK_OUT1: now also J5.3 (Pin_3)
- net BCLK_OUT1: now reaches U2.43 (BCLK_OUT1)
- net BCLK_OUT1: now also J5.2 (Pin_2)
- net SDATA_OUT1: now reaches U2.44 (SDATA_OUT1)
- net SDATA_OUT1: now also J5.5 (Pin_5)
- net LRCLK_OUT2: now reaches U2.47 (LRCLK_OUT2/MP8)
- net LRCLK_OUT2: now also J6.3 (Pin_3)
- net BCLK_OUT2: now reaches U2.48 (BCLK_OUT2)
- net BCLK_OUT2: now also J6.2 (Pin_2)
- net SDATA_OUT2: now reaches U2.49 (SDATA_OUT2)
- net SDATA_OUT2: now also J6.5 (Pin_5)
- net LRCLK_OUT3: now reaches U2.50 (LRCLK_OUT3/MP9)
- net LRCLK_OUT3: now also J7.3 (Pin_3)
- net BCLK_OUT3: now reaches U2.51 (BCLK_OUT3)
- net BCLK_OUT3: now also J7.2 (Pin_2)
- net SDATA_OUT3: now reaches U2.52 (SDATA_OUT3)
- net SDATA_OUT3: now also J7.5 (Pin_5)
- net SDATA_IN1: now reaches U2.62 (SDATA_IN1)
- net SDATA_IN1: now also J5.4 (Pin_4)
- net SDATA_IN2: now reaches U2.67 (SDATA_IN2)
- net SDATA_IN2: now also J6.4 (Pin_4)
- net SDATA_IN3: now reaches U2.70 (SDATA_IN3)
- net SDATA_IN3: now also J7.4 (Pin_4)
- no-connect marks 18 -> 24

Commit message: Assigned footprint.
Parts:
- C10, C12, C14, C15, C16, C17, C19, C20, C21, C22, C24, C25, C27, C28, C29, C30, C31, C38: footprint (none) -> Capacitor_SMD:C_0201_0603Metric
- C11, C13, C18, C23: footprint (none) -> Capacitor_SMD:C_0402_1005Metric
- Q3: footprint (none) -> Package_TO_SOT_SMD:TO-252-2
- R5, R6, R7, R9: footprint (none) -> Resistor_SMD:R_0201_0603Metric
- R8: footprint Resistor_SMD:R_0402_1005Metric -> Resistor_SMD:R_0201_0603Metric
- SW1: footprint (none) -> My_Parts:SKRPABE010
- U2: footprint CP_72_6_ADI -> My_Parts:CP_72_6_ADI
- U8: footprint (none) -> Package_TO_SOT_SMD:SOT-143
- X1: footprint (none) -> Oscillator:Oscillator_SMD_SeikoEpson_SG210-4Pin_2.5x2.0mm
Changed lines of the file:
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@@
 			)
 		)
-		(property "Footprint" ""
+		(property "Footprint" "Capacitor_SMD:C_0201_0603Metric"
 			(at 282.9052 184.15 0)
 			(effects
@@
 			)
 		)
-		(property "Footprint" ""
+		(property "Footprint" "Capacitor_SMD:C_0201_0603Metric"
 			(at 374.3452 184.15 0)
 			(effects
@@
 			)
 		)
-		(property "Footprint" ""
+		(property "Footprint" "Package_TO_SOT_SMD:SOT-143"
 			(at 76.2 147.32 0)
 			(effects
@@
 			)
 		)
-		(property "Footprint" ""
+		(property "Footprint" "Resistor_SMD:R_0201_0603Metric"
 			(at 89.408 157.48 90)
 			(effects
@@
 			)
 		)
-		(property "Footprint" ""
+		(property "Footprint" "Capacitor_SMD:C_0201_0603Metric"
 			(at 246.0752 184.15 0)
 			(effects
@@
 			)
 		)
-		(property "Footprint" ""
+		(property "Footprint" "Capacitor_SMD:C_0201_0603Metric"
 			(at 274.0152 184.15 0)
 			(effects
@@
 			)
 		)
-		(property "Footprint" ""
+		(property "Footprint" "Capacitor_SMD:C_0201_0603Metric"
 			(at 107.95 151.4348 0)
 			(effects
@@
 			)
 		)
-		(property "Footprint" ""
+		(property "Footprint" "Capacitor_SMD:C_0402_1005Metric"
 			(at 235.9152 184.15 0)
 			(effects
@@
 			)
 		)
-		(property "Footprint" ""
+		(property "Footprint" "My_Parts:SKRPABE010"
 			(at 104.14 139.7 0)
 			(effects
@@
 			)
 		)
-		(property "Footprint" "CP_72_6_ADI"
+		(property "Footprint" "My_Parts:CP_72_6_ADI"
 			(at 199.136 128.524 0)
 			(effects
@@
 			)
 		)
-		(property "Footprint" ""
+		(property "Footprint" "Capacitor_SMD:C_0201_0603Metric"
 			(at 347.6752 184.15 0)
 			(effects
@@
 			)
 		)
-		(property "Footprint" ""
+		(property "Footprint" "Capacitor_SMD:C_0402_1005Metric"
 			(at 254.9652 184.15 0)
 			(effects
@@
 			)
 		)
-		(property "Footprint" ""
+		(property "Footprint" "Capacitor_SMD:C_0201_0603Metric"
 			(at 227.0252 184.15 0)
 			(effects
@@
 			)
 		)
-		(property "Footprint" ""
+		(property "Footprint" "Capacitor_SMD:C_0201_0603Metric"
 			(at 300.6852 184.15 0)
 			(effects
@@
 			)
 		)
-		(property "Footprint" ""
+		(property "Footprint" "Capacitor_SMD:C_0201_0603Metric"
 			(at 108.9152 100.33 0)
 			(effects
@@
 			)
 		)
-		(property "Footprint" ""
+		(property "Footprint" "Capacitor_SMD:C_0201_0603Metric"
 			(at 309.5752 184.15 0)
 			(effects
@@
 			)
 		)
-		(property "Footprint" ""
+		(property "Footprint" "Oscillator:Oscillator_SMD_SeikoEpson_SG210-4Pin_2.5x2.0mm"
 			(at 87.63 203.2 0)
 			(effects
@@
 			)
 		)
-		(property "Footprint" ""
+		(property "Footprint" "Capacitor_SMD:C_0201_0603Metric"
 			(at 318.4652 184.15 0)
 			(effects
@@
 			)
 		)
-		(property "Footprint" "Resistor_SMD:R_0402_1005Metric"
+		(property "Footprint" "Resistor_SMD:R_0201_0603Metric"
 			(at 83.82 196.088 90)
 			(effects
@@
 			)
 		)
-		(property "Footprint" ""
+		(property "Footprint" "Capacitor_SMD:C_0201_0603Metric"
 			(at 365.4552 184.15 0)
 			(effects
@@
 			)
 		)
-		(property "Footprint" ""
+		(property "Footprint" "Capacitor_SMD:C_0201_0603Metric"
 			(at 356.5652 184.15 0)
 			(effects
@@
 			)
 		)
-		(property "Footprint" ""
+		(property "Footprint" "Resistor_SMD:R_0201_0603Metric"
 			(at 118.11 91.948 90)
 			(effects
@@
 			)
 		)
-		(property "Footprint" ""
+		(property "Footprint" "Capacitor_SMD:C_0201_0603Metric"
 			(at 327.3552 184.15 0)
 			(effects
@@
 			)
 		)
-		(property "Footprint" ""
+		(property "Footprint" "Capacitor_SMD:C_0402_1005Metric"
 			(at 336.2452 184.15 0)
 			(effects
@@
 			)
 		)
-		(property "Footprint" ""
+		(property "Footprint" "Capacitor_SMD:C_0201_0603Metric"
 			(at 56.8452 154.94 0)
 			(effects
@@
 			)
 		)
-		(property "Footprint" ""
+		(property "Footprint" "Capacitor_SMD:C_0402_1005Metric"
 			(at 383.2352 184.15 0)
 			(effects
@@
 			)
 		)
-		(property "Footprint" ""
+		(property "Footprint" "Capacitor_SMD:C_0201_0603Metric"
 			(at 265.1252 184.15 0)
 			(effects
@@
 			)
 		)
-		(property "Footprint" ""
+		(property "Footprint" "Resistor_SMD:R_0201_0603Metric"
 			(at 118.11 84.328 90)
 			(effects
@@
 			)
 		)
-		(property "Footprint" ""
+		(property "Footprint" "Capacitor_SMD:C_0201_0603Metric"
 			(at 291.7952 184.15 0)
 			(effects
@@
 			)
 		)
-		(property "Footprint" ""
+		(property "Footprint" "Resistor_SMD:R_0201_0603Metric"
 			(at 133.35 86.868 90)
 			(effects
@@
 			)
 		)
-		(property "Footprint" ""
+		(property "Footprint" "Package_TO_SOT_SMD:TO-252-2"
 			(at 109.22 72.39 0)
 			(effects
@@
 			)
 		)
-		(property "Footprint" ""
+		(property "Footprint" "Capacitor_SMD:C_0201_0603Metric"
 			(at 121.92 101.9048 0)
 			(effects

Commit message: Updated schematics.
Parts:
- removed SW1: SW_MEC_5G, My_Parts:SKRPABE010, symbol My_Parts:SW_MEC_5G
- added J5: Conn_01x06, My_Parts:PinHeader_1x06_P2.54mm_Vertical, symbol Connector_Generic:Conn_01x06
- added SW2: SKRPABE010, My_Parts:SKRPABE010, symbol Switch:SW_MEC_5E
- renumbered C25 to C36, C24 to C37, C27 to C38, C38 to C39, C10 to C40, C11 to C41, C12 to C42, C13 to C43, C28 to C44, C14 to C45, C29 to C46, C15 to C47, C30 to C48, C16 to C49, C31 to C50, C17 to C51, C18 to C52, C19 to C53, C20 to C54, C21 to C55, C22 to C56, C23 to C57, C26 to C58, J5 to J6, J6 to J7, J7 to J8, Q3 to Q1, R7 to R6, R6 to R7, R9 to R8, R8 to R9, U2 to U3, U8 to U4, X1 to X2
Connections:
- net 3V3: now also J5.1 (Pin_1)
- net DSP_MISO: now also J5.5 (Pin_5)
- net DSP_MOSI: now also J5.4 (Pin_4)
- net DSP_RESET: now also SW2.1, SW2.2
- net DSP_SCLK: now also J5.3 (Pin_3)
- net DSP_SS: now also J5.2 (Pin_2)
- net GND: now also J5.6 (Pin_6), SW2.3 (K), SW2.4 (A)

Commit message: Re-annotation.
Parts:
- removed J5, J6, J7, J8: Conn_01x06, My_Parts:PinHeader_1x06_P2.54mm_Vertical, symbol Connector_Generic:Conn_01x06
- added J5: Conn_02x07_Odd_Even, Connector_PinHeader_2.54mm:PinHeader_2x07_P2.54mm_Vertical, symbol Connector_Generic:Conn_02x07_Odd_Even
- added J6: 15910060, Connector_PinHeader_2.54mm:PinHeader_2x03_P2.54mm_Vertical, symbol Connector_Generic:Conn_02x03_Odd_Even
- renumbered C36 to C39, C37 to C40, C38 to C41, C39 to C42, C40 to C43, C41 to C44, C42 to C45, C43 to C46, C44 to C47, C45 to C48, C46 to C49, C47 to C50, C48 to C51, C49 to C52, C50 to C53, C51 to C54, C52 to C55, C53 to C56, C54 to C57, C55 to C58, C56 to C59, C57 to C60, C58 to C61, R6 to R10, R7 to R11, R8 to R12, R9 to R13, R5 to R9, SW2 to SW4
Connections:
- net 3V3: now also J5.1 (Pin_1), J5.2 (Pin_2), J6.1 (Pin_1)
- net BCLK_OUT1: now also J5.5 (Pin_5)
- net BCLK_OUT2: now also J5.6 (Pin_6)
- net DSP_CLKOUT: now also J5.3 (Pin_3), J5.4 (Pin_4)
- net DSP_MISO: now also J6.5 (Pin_5)
- net DSP_MOSI: now also J6.4 (Pin_4)
- net DSP_SCLK: now also J6.3 (Pin_3)
- net DSP_SS: now also J6.2 (Pin_2)
- net GND: now also J5.13 (Pin_13), J5.14 (Pin_14), J6.6 (Pin_6)
- net LRCLK_OUT1: now also J5.7 (Pin_7)
- net LRCLK_OUT2: now also J5.8 (Pin_8)
- net SDATA_IN1: now also J5.9 (Pin_9)
- net SDATA_IN2: now also J5.10 (Pin_10)
- net SDATA_OUT1: now also J5.11 (Pin_11)
- net SDATA_OUT2: now also J5.12 (Pin_12)
- net BCLK_OUT3: no longer names the net of U3.51 (BCLK_OUT3)
- net LRCLK_OUT3: no longer names the net of U3.50 (LRCLK_OUT3/MP9)
- net SDATA_IN3: no longer names the net of U3.70 (SDATA_IN3)
- net SDATA_OUT3: no longer names the net of U3.52 (SDATA_OUT3)
- no-connect marks 24 -> 28

Commit message: Change the order of IO assignment to pin headers.
Connections:
- net SDATA_IN1: now also J5.11 (Pin_11); no longer J5.9 (Pin_9)
- net SDATA_IN2: now also J5.12 (Pin_12); no longer J5.10 (Pin_10)
- net SDATA_OUT1: now also J5.9 (Pin_9); no longer J5.11 (Pin_11)
- net SDATA_OUT2: now also J5.10 (Pin_10); no longer J5.12 (Pin_12)
Changed lines of the file:
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@@
 		)
 	)
-	(label "SDATA_IN1"
+	(label "SDATA_OUT1"
 		(at 167.64 229.87 180)
 		(effects
@@
 		)
 	)
-	(label "SDATA_OUT1"
+	(label "SDATA_IN1"
 		(at 167.64 232.41 180)
 		(effects
@@
 		)
 	)
-	(label "SDATA_OUT2"
+	(label "SDATA_IN2"
 		(at 185.42 232.41 0)
 		(effects
@@
 		)
 	)
-	(label "SDATA_IN2"
+	(label "SDATA_OUT2"
 		(at 185.42 229.87 0)
 		(effects

Commit message: Modified wiring between ICs.
Changed lines of the file:
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@@
 	)
 	(hierarchical_label "DSP_LRCLK_IN0"
-		(shape input)
+		(shape output)
 		(at 157.48 140.97 180)
 		(effects
@@
 	)
 	(hierarchical_label "DSP_BCLK_IN0"
-		(shape input)
+		(shape output)
 		(at 157.48 118.11 180)
 		(effects

Commit message: Added some resistors and Schottky diode.
Parts:
- added R13, R14, R15, R16, R18, R19, R9: 33R, Resistor_SMD:R_0201_0603Metric, symbol Device:R
- added R25: 10k, Resistor_SMD:R_0201_0603Metric, symbol Device:R
- renumbered R9 to R10, R10 to R11, R11 to R12, R12 to R17, R13 to R20
Connections:
- net 3V3: now also R25.2
- net DSP_BCLK_IN0: now also R13.1; no longer U3.57 (BCLK_IN0)
- net DSP_BCLK_OUT0: now also R14.1; no longer U3.40 (BCLK_OUT0)
- net DSP_CLKOUT: now also R9.2; no longer U3.23 (CLKOUT)
- net DSP_LRCLK_IN0: now also R15.1; no longer U3.58 (LRCLK_IN0/MP10)
- net DSP_LRCLK_OUT0: now also R16.1; no longer U3.39 (LRCLK_OUT0/MP4)
- net DSP_SDATA_IN0: now also R18.1; no longer U3.59 (SDATA_IN0)
- net DSP_SDATA_OUT0: now also R19.1; no longer U3.41 (SDATA_OUT0)
- net DSP_SS: now also R25.1
- new net: R18.2, U3.59 (SDATA_IN0)
- new net: R9.1, U3.23 (CLKOUT)
- new net: R16.2, U3.39 (LRCLK_OUT0/MP4)
- new net: R14.2, U3.40 (BCLK_OUT0)
- new net: R19.2, U3.41 (SDATA_OUT0)
- new net: R13.2, U3.57 (BCLK_IN0)
- new net: R15.2, U3.58 (LRCLK_IN0/MP10)
