File: KiCad/OTO_NO_ITA/dsp.kicad_sch (KiCad schematic)
At the start: 43 parts, among them J5 Conn_02x07_Odd_Even, J6 15910060, Q1 STD2805T4, SW4 SKRPABE010, U3 ADAU1466WBCPZ300RL, U4 ADM811TARTZ, X2 12.288MHz

Commit message: Modified the pin header J6 for USBi.
Parts:
- removed J6: 15910060, Connector_PinHeader_2.54mm:PinHeader_2x03_P2.54mm_Vertical, symbol Connector_Generic:Conn_02x03_Odd_Even
- added D7: LED, LED_SMD:LED_0603_1608Metric, symbol Device:LED
- added J6: Conn_02x04_Odd_Even, Connector_PinHeader_2.54mm:PinHeader_2x04_P2.54mm_Vertical, symbol Connector_Generic:Conn_02x04_Odd_Even
- added R26: 1k, Resistor_SMD:R_0201_0603Metric, symbol Device:R
Connections:
- net DSP_MISO: now also J6.3 (Pin_3)
- net DSP_MOSI: now also J6.6 (Pin_6)
- net DSP_SCLK: now also J6.5 (Pin_5)
- net DSP_SS: now also J6.7 (Pin_7)
- net GND: now also D7.1 (K), J6.8 (Pin_8)
- new net: J6.2 (Pin_2), R26.1
- new net: D7.2 (A), R26.2
- no-connect marks 28 -> 30

Commit message: Changed pin assignments for J4 and J6.
Parts:
- J5: footprint Connector_PinHeader_2.54mm:PinHeader_2x07_P2.54mm_Vertical -> Connector_PinSocket_2.54mm:PinSocket_2x07_P2.54mm_Vertical
Connections:
- net BCLK_OUT1: now also J5.6 (Pin_6); no longer J5.5 (Pin_5)
- net BCLK_OUT2: now also J5.5 (Pin_5); no longer J5.6 (Pin_6)
- net LRCLK_OUT1: now also J5.8 (Pin_8); no longer J5.7 (Pin_7)
- net LRCLK_OUT2: now also J5.7 (Pin_7); no longer J5.8 (Pin_8)
- net SDATA_IN1: now also J5.12 (Pin_12); no longer J5.11 (Pin_11)
- net SDATA_IN2: now also J5.11 (Pin_11); no longer J5.12 (Pin_12)
- net SDATA_OUT1: now also J5.10 (Pin_10); no longer J5.9 (Pin_9)
- net SDATA_OUT2: now also J5.9 (Pin_9); no longer J5.10 (Pin_10)
Changed lines of the file:
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@@
-	(wire
-		(pts
-			(xy 167.64 227.33) (xy 170.18 227.33)
-		)
-		(stroke
-			(width 0)
-			(type default)
-		)
-	)
 	(wire
 		(pts
@@
 	(wire
 		(pts
-			(xy 167.64 232.41) (xy 170.18 232.41)
-		)
-		(stroke
-			(width 0)
-			(type default)
-		)
-	)
-	(wire
-		(pts
 			(xy 273.05 184.15) (xy 273.05 186.69)
 		)
@@
 	(wire
 		(pts
-			(xy 170.18 234.95) (xy 163.83 234.95)
-		)
-		(stroke
-			(width 0)
-			(type default)
-		)
-	)
-	(wire
-		(pts
 			(xy 124.46 102.87) (xy 124.46 90.17)
 		)
@@
 	(wire
 		(pts
-			(xy 167.64 224.79) (xy 170.18 224.79)
-		)
-		(stroke
-			(width 0)
-			(type default)
-		)
-	)
-	(wire
-		(pts
 			(xy 138.43 151.13) (xy 143.51 151.13)
 		)
@@
 	(wire
 		(pts
+			(xy 163.83 234.95) (xy 170.18 234.95)
+		)
+		(stroke
+			(width 0)
+			(type default)
+		)
+	)
+	(wire
+		(pts
 			(xy 85.09 151.13) (xy 87.63 151.13)
 		)
@@
 	(wire
 		(pts
+			(xy 170.18 222.25) (xy 167.64 222.25)
+		)
+		(stroke
+			(width 0)
+			(type default)
+		)
+	)
+	(wire
+		(pts
 			(xy 373.38 184.15) (xy 373.38 186.69)
 		)
@@
 	(wire
 		(pts
-			(xy 167.64 229.87) (xy 170.18 229.87)
-		)
-		(stroke
-			(width 0)
-			(type default)
-		)
-	)
-	(wire
-		(pts
 			(xy 151.13 118.11) (xy 162.56 118.11)
 		)
@@
 	(wire
 		(pts
-			(xy 167.64 222.25) (xy 170.18 222.25)
-		)
-		(stroke
-			(width 0)
-			(type default)
-		)
-	)
-	(wire
-		(pts
 			(xy 107.95 90.17) (xy 107.95 92.71)
 		)
@@
 	)
 	(label "SDATA_OUT1"
-		(at 167.64 229.87 180)
+		(at 170.18 229.87 180)
 		(effects
 			(font
@@
 	)
 	(label "CLKOUT"
-		(at 167.64 222.25 180)
+		(at 170.18 222.25 180)
 		(effects
 			(font
@@
 	)
 	(label "SDATA_IN1"
-		(at 167.64 232.41 180)
+		(at 170.18 232.41 180)
 		(effects
 			(font
@@
 	)
 	(label "BCLK_OUT1"
-		(at 167.64 224.79 180)
+		(at 170.18 224.79 180)
 		(effects
 			(font
@@
 	)
 	(label "LRCLK_OUT1"
-		(at 167.64 227.33 180)
+		(at 170.18 227.33 180)
 		(effects
 			(font
@@
 	(symbol
 		(lib_id "Connector_Generic:Conn_02x07_Odd_Even")
-		(at 175.26 227.33 0)
+		(at 177.8 227.33 0)
+		(mirror y)
 		(unit 1)
 		(exclude_from_sim no)
@@
 		(dnp no)
 		(property "Reference" "J5"
-			(at 176.276 217.17 0)
+			(at 176.784 217.17 0)
 			(effects
 				(font
@@
 		)
 		(property "Value" "Conn_02x07_Odd_Even"
-			(at 176.276 237.744 0)
-			(effects
-				(font
-					(size 1.27 1.27)
-				)
-			)
-		)
-		(property "Footprint" "Connector_PinHeader_2.54mm:PinHeader_2x07_P2.54mm_Vertical"
-			(at 175.26 227.33 0)
+			(at 176.784 237.744 0)
+			(effects
+				(font
+					(size 1.27 1.27)
+				)
+			)
+		)
+		(property "Footprint" "Connector_PinSocket_2.54mm:PinSocket_2x07_P2.54mm_Vertical"
+			(at 177.8 227.33 0)
 			(effects
 				(font
@@
 		)
 		(property "Datasheet" "~"
-			(at 175.26 227.33 0)
+			(at 177.8 227.33 0)
 			(effects
 				(font
@@
 		)
 		(property "Description" "Generic connector, double row, 02x07, odd/even pin numbering scheme (row 1 odd numbers, row 2 even numbers), script generated (kicad-library-utils/schlib/autogen/connector/)"
-			(at 175.26 227.33 0)
-			(effects
-				(font
+			(at 177.8 227.33 0)
+			(effects
+				(font
