File: KiCad/OTO_NO_ITA/usb.kicad_sch (KiCad schematic)
At the start: 4 parts, among them Q1 STL40DN3LLH5, Q2 STL40DN3LLH5, U3 TCPP03-M20, U4 ECMF2-40A100N6

Commit message: Updated schematics.
Parts:
- added C1: 2.2uF/50V, symbol Device:C
- added C2: 100nF, symbol Device:C
- added C3, C4: 560pF, symbol Device:C
- added J4: UB1611-HGN, My_Parts:Gangyuan_UB1611-HGN, symbol My_Parts:5077CR-16SMC2-BK-TR
- added R1, R3: 10k, symbol Device:R
- added R2: 22mR, symbol Device:R
- added R4: 2k4, symbol Device:R
- added U6: ESDA25P35-1U1M, symbol My_Parts:ESDA25P35-1U1M
Connections:
- net UCPD_CC1: now reaches U3.1 (CC1)
- net at U3.10 (I_SENSE): now also Q1.7 (D2), Q1.8 (D2), Q2.7 (D2), Q2.8 (D2), R2.1
- net at U3.11 (V_SENSE): now also R3.2, R4.1
- net GND: now reaches U3.12 (GND)
- net GND: now also U3.21 (GND), U4.3 (GND), U4.4 (GND), C1.2, C2.2, C3.2, C4.2, J4.A1_B12 (GND), J4.B1_A12 (GND), J4.S1 (SHIELD), J4.S2 (SHIELD), J4.S3 (SHIELD), J4.S4 (SHIELD), R1.2, R4.2, U6.2
- net CC2: now reaches U3.13 (CC_2c)
- net CC2: now also C3.1, J4.B5 (CC2)
- net at U3.14 (C_BIAS): now also C2.1
- net CC1: now reaches U3.15 (CC_1c)
- net CC1: now also C4.1, J4.A5 (CC1)
- net at U3.16 (I2C_ADD): now also R1.1
- net UCPD_SDA: now reaches U3.17 (SDA)
- net UCPD_SCL: now reaches U3.18 (SCL)
- net UCPD_INT: now reaches U3.19 (FLG_n)
- net 3V3: now reaches U3.2 (VCC_VCONN)
- net UCPD_PWR_EN: now reaches U3.20 (EN)
- net UCPD_CC2: now reaches U3.3 (CC2)
- net UCPD_ISENSE: now reaches U3.4 (I_ANA)
- net at U3.5 (GDP_g): now also Q2.2 (G2), Q2.4 (G1)
- net at U3.6 (GDP_s): now also Q2.1 (S2), Q2.3 (S1)
- net at U3.7 (GDC_g): now also Q1.2 (G2), Q1.4 (G1)
- net at U3.8 (GDC_s): now also Q1.1 (S2), Q1.3 (S1)
- net VBUS: now reaches U3.9 (VBUS_c)
- net VBUS: now also C1.1, J4.A4_B9 (VBUS), J4.B4_A9 (VBUS), R2.2, R3.1, U6.1
- net 5V_UCPD: now reaches Q1.5 (D1)
- net 5V_UCPD: now also Q1.6 (D1)
- net 5V: now reaches Q2.5 (D1)
- net 5V: now also Q2.6 (D1)
- net D+: now reaches U4.1 (D+_con)
- net D+: now also J4.A6 (DP1), J4.B6 (DP2)
- net D-: now reaches U4.2 (D-_con)
- net D-: now also J4.A7 (DN1), J4.B7 (DN2)
- net USB_HS_D-: now reaches U4.5 (D-_ic)
- net USB_HS_D+: now reaches U4.6 (D+_ic)
- no-connect marks 0 -> 2
Other:
- note added: "diff pair 90ohm"
- moved on the sheet: Q1, Q2, U3, U4

Commit message: Updated schematics.
Changed lines of the file:
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@@
 	)
 	(hierarchical_label "UCPD_ISENSE"
-		(shape input)
+		(shape output)
 		(at 78.74 95.25 180)
 		(effects

Commit message: Assigned footprint.
Parts:
- C1: footprint (none) -> Capacitor_SMD:C_0603_1608Metric
- C2, C3, C4: footprint (none) -> Capacitor_SMD:C_0201_0603Metric
- Q1, Q2: footprint (none) -> My_Parts:SON_DN3LLH5_STM
- R1, R2, R3, R4: footprint (none) -> Resistor_SMD:R_0201_0603Metric
- U3: footprint (none) -> My_Parts:QFN-20L_4.0X4.0X0.75_STM
- U4: footprint (none) -> My_Parts:QFN6L_ECMF2_STM
- U6: footprint (none) -> My_Parts:QFN1610_STM
Changed lines of the file:
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@@
 			)
 		)
-		(property "Footprint" ""
+		(property "Footprint" "Capacitor_SMD:C_0201_0603Metric"
 			(at 139.3952 114.3 0)
 			(effects
@@
 			)
 		)
-		(property "Footprint" ""
+		(property "Footprint" "My_Parts:QFN-20L_4.0X4.0X0.75_STM"
 			(at 106.68 97.79 0)
 			(effects
@@
 			)
 		)
-		(property "Footprint" ""
+		(property "Footprint" "My_Parts:SON_DN3LLH5_STM"
 			(at 113.03 35.56 0)
 			(effects
@@
 			)
 		)
-		(property "Footprint" ""
+		(property "Footprint" "Resistor_SMD:R_0201_0603Metric"
 			(at 153.67 93.218 90)
 			(effects
@@
 			)
 		)
-		(property "Footprint" ""
+		(property "Footprint" "Capacitor_SMD:C_0201_0603Metric"
 			(at 130.5052 115.57 0)
 			(effects
@@
 			)
 		)
-		(property "Footprint" ""
+		(property "Footprint" "Resistor_SMD:R_0201_0603Metric"
 			(at 166.37 93.218 90)
 			(effects
@@
 			)
 		)
-		(property "Footprint" ""
+		(property "Footprint" "Resistor_SMD:R_0201_0603Metric"
 			(at 121.412 118.11 90)
 			(effects
@@
 			)
 		)
-		(property "Footprint" ""
+		(property "Footprint" "My_Parts:QFN1610_STM"
 			(at 238.76 106.68 0)
 			(effects
@@
 			)
 		)
-		(property "Footprint" ""
+		(property "Footprint" "My_Parts:SON_DN3LLH5_STM"
 			(at 121.92 64.77 0)
 			(effects
@@
 			)
 		)
-		(property "Footprint" ""
+		(property "Footprint" "Resistor_SMD:R_0201_0603Metric"
 			(at 140.97 57.658 90)
 			(effects
@@
 			)
 		)
-		(property "Footprint" ""
+		(property "Footprint" "Capacitor_SMD:C_0201_0603Metric"
 			(at 148.2852 114.3 0)
 			(effects
@@
 			)
 		)
-		(property "Footprint" ""
+		(property "Footprint" "Capacitor_SMD:C_0603_1608Metric"
 			(at 263.8552 109.22 0)
 			(effects
@@
 			)
 		)
-		(property "Footprint" ""
+		(property "Footprint" "My_Parts:QFN6L_ECMF2_STM"
 			(at 132.08 161.29 0)
 			(effects

Commit message: Updated schematics.
Parts:
- renumbered C1 to C65, C3 to C66, C4 to C67, C2 to C68, J4 to J9, Q1 to Q2, Q2 to Q3, R2 to R10, R3 to R11, R4 to R12, R1 to R13, U3 to U7, U6 to U8, U4 to U9
Changed lines of the file:
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@@
 		(on_board yes)
 		(dnp no)
-		(property "Reference" "#PWR01"
+		(property "Reference" "#PWR074"
 			(at 262.89 97.79 0)
 			(effects
@@
 			(project ""
 				(path "/9c594957-fd6c-4305-bab8-fba79a4c5d5c/48251e43-7df4-4aa3-bd6f-892bea7e5ba1"
-					(reference "#PWR01")
+					(reference "#PWR074")
 					(unit 1)
 				)
@@
 		(on_board yes)
 		(dnp no)
-		(property "Reference" "C3"
+		(property "Reference" "C66"
 			(at 140.716 110.49 0)
 			(effects
@@
 			(project "OTO_NO_ITA"
 				(path "/9c594957-fd6c-4305-bab8-fba79a4c5d5c/48251e43-7df4-4aa3-bd6f-892bea7e5ba1"
-					(reference "C3")
+					(reference "C66")
 					(unit 1)
 				)
@@
 		(on_board yes)
 		(dnp no)
-		(property "Reference" "U3"
+		(property "Reference" "U7"
 			(at 118.11 79.756 0)
 			(effects
@@
 			(project ""
 				(path "/9c594957-fd6c-4305-bab8-fba79a4c5d5c/48251e43-7df4-4aa3-bd6f-892bea7e5ba1"
-					(reference "U3")
+					(reference "U7")
 					(unit 1)
 				)
@@
 		(on_board yes)
 		(dnp no)
-		(property "Reference" "Q1"
+		(property "Reference" "Q2"
 			(at 105.41 40.386 0)
 			(effects
@@
 			(project ""
 				(path "/9c594957-fd6c-4305-bab8-fba79a4c5d5c/48251e43-7df4-4aa3-bd6f-892bea7e5ba1"
-					(reference "Q1")
+					(reference "Q2")
 					(unit 1)
 				)
@@
 		(on_board yes)
 		(dnp no)
-		(property "Reference" "R3"
+		(property "Reference" "R11"
 			(at 153.67 89.408 90)
 			(effects
@@
 			(project "OTO_NO_ITA"
 				(path "/9c594957-fd6c-4305-bab8-fba79a4c5d5c/48251e43-7df4-4aa3-bd6f-892bea7e5ba1"
-					(reference "R3")
+					(reference "R11")
 					(unit 1)
 				)
@@
 		(on_board yes)
 		(dnp no)
-		(property "Reference" "#PWR06"
+		(property "Reference" "#PWR077"
 			(at 138.43 125.73 0)
 			(effects
@@
 			(project "OTO_NO_ITA"
 				(path "/9c594957-fd6c-4305-bab8-fba79a4c5d5c/48251e43-7df4-4aa3-bd6f-892bea7e5ba1"
-					(reference "#PWR06")
+					(reference "#PWR077")
 					(unit 1)
 				)
@@
 		(on_board yes)
 		(dnp no)
-		(property "Reference" "#PWR012"
+		(property "Reference" "#PWR069"
 			(at 105.41 25.4 0)
 			(effects
@@
 			(project "OTO_NO_ITA"
 				(path "/9c594957-fd6c-4305-bab8-fba79a4c5d5c/48251e43-7df4-4aa3-bd6f-892bea7e5ba1"
-					(reference "#PWR012")
+					(reference "#PWR069")
 					(unit 1)
 				)
@@
 		(on_board yes)
 		(dnp no)
-		(property "Reference" "C2"
+		(property "Reference" "C68"
 			(at 131.826 111.76 0)
 			(effects
@@
 			(project "OTO_NO_ITA"
 				(path "/9c594957-fd6c-4305-bab8-fba79a4c5d5c/48251e43-7df4-4aa3-bd6f-892bea7e5ba1"
-					(reference "C2")
+					(reference "C68")
 					(unit 1)
 				)
@@
 		(on_board yes)
 		(dnp no)
-		(property "Reference" "R4"
+		(property "Reference" "R12"
 			(at 166.37 89.408 90)
 			(effects
@@
 			(project "OTO_NO_ITA"
 				(path "/9c594957-fd6c-4305-bab8-fba79a4c5d5c/48251e43-7df4-4aa3-bd6f-892bea7e5ba1"
-					(reference "R4")
+					(reference "R12")
 					(unit 1)
 				)
@@
 		(on_board yes)
 		(dnp no)
-		(property "Reference" "#PWR013"
+		(property "Reference" "#PWR072"
 			(at 90.17 88.9 0)
 			(effects
@@
 			(project "OTO_NO_ITA"
 				(path "/9c594957-fd6c-4305-bab8-fba79a4c5d5c/48251e43-7df4-4aa3-bd6f-892bea7e5ba1"
-					(reference "#PWR013")
+					(reference "#PWR072")
 					(unit 1)
 				)
@@
 		(on_board yes)
 		(dnp no)
-		(property "Reference" "J4"
+		(property "Reference" "J9"
 			(at 198.12 92.71 0)
 			(effects
@@
 			(project "OTO_NO_ITA"
 				(path "/9c594957-fd6c-4305-bab8-fba79a4c5d5c/48251e43-7df4-4aa3-bd6f-892bea7e5ba1"
-					(reference "J4")
+					(reference "J9")
 					(unit 1)
 				)
@@
 		(on_board yes)
 		(dnp no)
-		(property "Reference" "R1"
+		(property "Reference" "R13"
 			(at 124.46 117.094 0)
 			(effects
@@
 			(project ""
 				(path "/9c594957-fd6c-4305-bab8-fba79a4c5d5c/48251e43-7df4-4aa3-bd6f-892bea7e5ba1"
-					(reference "R1")
+					(reference "R13")
 					(unit 1)
 				)
@@
 		(on_board yes)
 		(dnp no)
-		(property "Reference" "U6"
+		(property "Reference" "U8"
 			(at 241.3 102.616 90)
 			(effects
@@
 			(project ""
 				(path "/9c594957-fd6c-4305-bab8-fba79a4c5d5c/48251e43-7df4-4aa3-bd6f-892bea7e5ba1"
-					(reference "U6")
+					(reference "U8")
 					(unit 1)
 				)
@@
 		(on_board yes)
 		(dnp no)
-		(property "Reference" "Q2"
+		(property "Reference" "Q3"
 			(at 114.046 69.596 0)
 			(effects
@@
 			(project ""
 				(path "/9c594957-fd6c-4305-bab8-fba79a4c5d5c/48251e43-7df4-4aa3-bd6f-892bea7e5ba1"
-					(reference "Q2")
+					(reference "Q3")
 					(unit 1)
 				)
@@
 		(on_board yes)
 		(dnp no)
-		(property "Reference" "#PWR07"
+		(property "Reference" "#PWR081"
 			(at 116.84 158.75 0)
 			(effects
@@
 			(project "OTO_NO_ITA"
 				(path "/9c594957-fd6c-4305-bab8-fba79a4c5d5c/48251e43-7df4-4aa3-bd6f-892bea7e5ba1"
-					(reference "#PWR07")
+					(reference "#PWR081")
 					(unit 1)
 				)
@@
 		(on_board yes)
 		(dnp no)
-		(property "Reference" "#PWR02"
+		(property "Reference" "#PWR076"
 			(at 262.89 123.19 0)
 			(effects
@@
 			(project ""
 				(path "/9c594957-fd6c-4305-bab8-fba79a4c5d5c/48251e43-7df4-4aa3-bd6f-892bea7e5ba1"
-					(reference "#PWR02")
+					(reference "#PWR076")
 					(unit 1)
 				)
@@
 		(on_board yes)
 		(dnp no)
-		(property "Reference" "#PWR010"
+		(property "Reference" "#PWR071"
 			(at 147.32 57.15 0)
 			(effects
@@
 			(project "OTO_NO_ITA"
 				(path "/9c594957-fd6c-4305-bab8-fba79a4c5d5c/48251e43-7df4-4aa3-bd6f-892bea7e5ba1"
-					(reference "#PWR010")
+					(reference "#PWR071")
 					(unit 1)
 				)
@@
 		(on_board yes)
 		(dnp no)
-		(property "Reference" "#PWR08"
+		(property "Reference" "#PWR080"
 			(at 96.52 158.75 0)
 			(effects
@@
 			(project "OTO_NO_ITA"
 				(path "/9c594957-fd6c-4305-bab8-fba79a4c5d5c/48251e43-7df4-4aa3-bd6f-892bea7e5ba1"
-					(reference "#PWR08")
+					(reference "#PWR080")
 					(unit 1)
 				)
@@
 		(on_board yes)
 		(dnp no)
-		(property "Reference" "#PWR05"
+		(property "Reference" "#PWR079"
 			(at 129.54 132.08 0)
 			(effects
@@
 			(project "OTO_NO_ITA"
 				(path "/9c594957-fd6c-4305-bab8-fba79a4c5d5c/48251e43-7df4-4aa3-bd6f-892bea7e5ba1"
-					(reference "#PWR05")
+					(reference "#PWR079")
 					(unit 1)
 				)
@@
 		(on_board yes)
 		(dnp no)
-		(property "Reference" "R2"
+		(property "Reference" "R10"
 			(at 140.97 53.848 90)
 			(effects
@@
 			(project "OTO_NO_ITA"
 				(path "/9c594957-fd6c-4305-bab8-fba79a4c5d5c/48251e43-7df4-4aa3-bd6f-892bea7e5ba1"
-					(reference "R2")
+					(reference "R10")
 					(unit 1)
 				)
@@
 		(on_board yes)
 		(dnp no)
-		(property "Reference" "#PWR09"
+		(property "Reference" "#PWR070"
 			(at 114.3 54.61 0)
 			(effects
@@
 			(project "OTO_NO_ITA"
 				(path "/9c594957-fd6c-4305-bab8-fba79a4c5d5c/48251e43-7df4-4aa3-bd6f-892bea7e5ba1"
-					(reference "#PWR09")
+					(reference "#PWR070")
 					(unit 1)
 				)
@@
 		(on_board yes)
 		(dnp no)
-		(property "Reference" "C4"
+		(property "Reference" "C67"
 			(at 149.606 110.49 0)
 			(effects
@@
 			(project "OTO_NO_ITA"
 				(path "/9c594957-fd6c-4305-bab8-fba79a4c5d5c/48251e43-7df4-4aa3-bd6f-892bea7e5ba1"
-					(reference "C4")
+					(reference "C67")
 					(unit 1)
 				)
@@
 		(dnp no)
 		(fields_autoplaced yes)
-		(property "Reference" "C1"
+		(property "Reference" "C65"
 			(at 266.7 104.1399 0)
 			(effects
@@
 			(project ""
 				(path "/9c594957-fd6c-4305-bab8-fba79a4c5d5c/48251e43-7df4-4aa3-bd6f-892bea7e5ba1"
-					(reference "C1")
+					(reference "C65")
 					(unit 1)
 				)
@@
 		(on_board yes)
 		(dnp no)
-		(property "Reference" "#PWR04"
+		(property "Reference" "#PWR078"
 			(at 105.41 132.08 0)
 			(effects
@@
 			(project "OTO_NO_ITA"
 				(path "/9c594957-fd6c-4305-bab8-fba79a4c5d5c/48251e43-7df4-4aa3-bd6f-892bea7e5ba1"
-					(reference "#PWR04")
+					(reference "#PWR078")
 					(unit 1)
 				)
@@
 		(on_board yes)
 		(dnp no)
-		(property "Reference" "U4"
+		(property "Reference" "U9"
 			(at 106.68 135.89 0)
 			(effects
@@
 			(project ""
 				(path "/9c594957-fd6c-4305-bab8-fba79a4c5d5c/48251e43-7df4-4aa3-bd6f-892bea7e5ba1"
-					(reference "U4")
+					(reference "U9")
 					(unit 1)
 				)
@@
 		(on_board yes)
 		(dnp no)
-		(property "Reference" "#PWR03"
+		(property "Reference" "#PWR075"
 			(at 191.77 123.19 0)
 			(effects
@@
 			(project "OTO_NO_ITA"
 				(path "/9c594957-fd6c-4305-bab8-fba79a4c5d5c/48251e43-7df4-4aa3-bd6f-892bea7e5ba1"
-					(reference "#PWR03")
+					(reference "#PWR075")
 					(unit 1)
 				)
@@
 		(on_board yes)
 		(dnp no)
-		(property "Reference" "#PWR011"
+		(property "Reference" "#PWR073"
 			(at 179.07 91.44 0)
 			(effects
@@
 			(project "OTO_NO_ITA"
 				(path "/9c594957-fd6c-4305-bab8-fba79a4c5d5c/48251e43-7df4-4aa3-bd6f-892bea7e5ba1"
-					(reference "#PWR011")
-					(unit 1)
-				)
+					(reference "#PWR073")
+					(unit 1)
+				)

Commit message: Re-annotation.
Parts:
- added D5: D_Schottky, Diode_SMD:D_PowerDI-123, symbol Device:D_Schottky
- added J7, J8: Conn_01x02, Connector_PinHeader_2.54mm:PinHeader_1x02_P2.54mm_Vertical, symbol Connector_Generic:Conn_01x02
- renumbered C65 to C68, C66 to C69, C67 to C70, C68 to C71, R10 to R14, R11 to R15, R12 to R16, R13 to R17
Connections:
- net 5V: now also J8.1 (Pin_1)
- net 5V_UCPD: now also D5.1 (K)
- net GND: now also J7.2 (Pin_2), J8.2 (Pin_2)
- new net: D5.2 (A), J7.1 (Pin_1)
Other:
- note added: "SINK"
- note added: "SOURCE"

Commit message: Changed the footprint size of R14.
Parts:
- R14: footprint Resistor_SMD:R_0201_0603Metric -> Resistor_SMD:R_0603_1608Metric
Changed lines of the file:
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@@
 			)
 		)
-		(property "Footprint" "Resistor_SMD:R_0201_0603Metric"
+		(property "Footprint" "Resistor_SMD:R_0603_1608Metric"
 			(at 140.97 57.658 90)
 			(effects

Commit message: Added some resistors and Schottky diode.
Parts:
- renumbered R14 to R21, R15 to R22, R16 to R23, R17 to R24
Changed lines of the file:
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@@
 		(on_board yes)
 		(dnp no)
-		(property "Reference" "R15"
+		(property "Reference" "R22"
 			(at 153.67 89.408 90)
 			(effects
@@
 			(project "OTO_NO_ITA"
 				(path "/9c594957-fd6c-4305-bab8-fba79a4c5d5c/48251e43-7df4-4aa3-bd6f-892bea7e5ba1"
-					(reference "R15")
+					(reference "R22")
 					(unit 1)
 				)
@@
 		(on_board yes)
 		(dnp no)
-		(property "Reference" "R16"
+		(property "Reference" "R23"
 			(at 166.37 89.408 90)
 			(effects
@@
 			(project "OTO_NO_ITA"
 				(path "/9c594957-fd6c-4305-bab8-fba79a4c5d5c/48251e43-7df4-4aa3-bd6f-892bea7e5ba1"
-					(reference "R16")
+					(reference "R23")
 					(unit 1)
 				)
@@
 		(on_board yes)
 		(dnp no)
-		(property "Reference" "R17"
+		(property "Reference" "R24"
 			(at 124.46 117.094 0)
 			(effects
@@
 			(project ""
 				(path "/9c594957-fd6c-4305-bab8-fba79a4c5d5c/48251e43-7df4-4aa3-bd6f-892bea7e5ba1"
-					(reference "R17")
+					(reference "R24")
 					(unit 1)
 				)
@@
 		(on_board yes)
 		(dnp no)
-		(property "Reference" "R14"
+		(property "Reference" "R21"
 			(at 140.97 53.848 90)
 			(effects
@@
 			(project "OTO_NO_ITA"
 				(path "/9c594957-fd6c-4305-bab8-fba79a4c5d5c/48251e43-7df4-4aa3-bd6f-892bea7e5ba1"
-					(reference "R14")
-					(unit 1)
-				)
+					(reference "R21")
+					(unit 1)
+				)

Commit message: Change J7 and J8(5V in/out connector) to JST PH.
Parts:
- J7, J8: footprint Connector_PinHeader_2.54mm:PinHeader_1x02_P2.54mm_Vertical -> Connector_JST:JST_PH_S2B-PH-K_1x02_P2.00mm_Horizontal
Changed lines of the file:
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@@
 			)
 		)
-		(property "Footprint" "Connector_PinHeader_2.54mm:PinHeader_1x02_P2.54mm_Vertical"
+		(property "Footprint" "Connector_JST:JST_PH_S2B-PH-K_1x02_P2.00mm_Horizontal"
 			(at 238.76 46.99 0)
 			(effects
@@
 			)
 		)
-		(property "Footprint" "Connector_PinHeader_2.54mm:PinHeader_1x02_P2.54mm_Vertical"
+		(property "Footprint" "Connector_JST:JST_PH_S2B-PH-K_1x02_P2.00mm_Horizontal"
 			(at 187.96 46.99 0)
 			(effects
