File: KiCad/OTO_NO_ITA/usb.kicad_sch (KiCad schematic)
At the start: 17 parts, among them J7 Conn_01x02, J8 Conn_01x02, J9 UB1611-HGN, Q2 STL40DN3LLH5, Q3 STL40DN3LLH5, U7 TCPP03-M20, U8 ESDA25P35-1U1M, U9 ECMF2-40A100N6

Commit message: Fixed some mistakes.
switched 5V and 5V_UCPD.
switched VREFP and VREFM.
Connections:
- net 5V: now also D5.1 (K); no longer J8.1 (Pin_1)
- net 5V_UCPD: now also J8.1 (Pin_1); no longer D5.1 (K)
Changed lines of the file:
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@@
 			)
 		)
-		(property "Value" "5V"
+		(property "Value" "5V_UCPD"
 			(at 231.14 40.64 0)
 			(effects
@@
 			)
 		)
-		(property "Value" "5V_UCPD"
+		(property "Value" "5V"
 			(at 208.28 40.64 0)
 			(effects
