File: KiCad/OTO_NO_ITA/OTO_NO_ITA.kicad_sch (KiCad schematic)
At the start: 0 parts

Commit message: Updated schematics.
Other:
- sheet DSP ports: added DSP_BCLK_IN0, DSP_BCLK_OUT0, DSP_CLKOUT, DSP_LRCLK_IN0, DSP_LRCLK_OUT0, DSP_MISO, DSP_MOSI, DSP_RESET, DSP_SCLK, DSP_SDATA_IN0, DSP_SDATA_OUT0, DSP_SS; removed none
- sheet USB ports: added UCPD_CC1, UCPD_CC2, UCPD_INT, UCPD_ISENSE, UCPD_PWR_EN, UCPD_SCL, UCPD_SDA, USB_HS_D+, USB_HS_D-; removed none
Changed lines of the file:
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@@
 	(paper "A4")
 	(sheet
-		(at 167.64 111.76)
-		(size 72.39 44.45)
+		(at 210.82 91.44)
+		(size 24.13 44.45)
 		(exclude_from_sim no)
 		(in_bom yes)
@@
 		)
 		(property "Sheetname" "USB"
-			(at 167.64 111.0484 0)
+			(at 210.82 90.7284 0)
 			(effects
 				(font
@@
 		)
 		(property "Sheetfile" "usb.kicad_sch"
-			(at 167.64 156.7946 0)
+			(at 210.82 136.4746 0)
 			(effects
 				(font
@@
 				)
 				(justify left top)
+			)
+		)
+		(pin "UCPD_PWR_EN" input
+			(at 210.82 96.52 180)
+			(effects
+				(font
+					(size 1.27 1.27)
+				)
+				(justify left)
+			)
+		)
+		(pin "UCPD_CC1" bidirectional
+			(at 210.82 104.14 180)
+			(effects
+				(font
+					(size 1.27 1.27)
+				)
+				(justify left)
+			)
+		)
+		(pin "UCPD_ISENSE" input
+			(at 210.82 111.76 180)
+			(effects
+				(font
+					(size 1.27 1.27)
+				)
+				(justify left)
+			)
+		)
+		(pin "UCPD_CC2" bidirectional
+			(at 210.82 106.68 180)
+			(effects
+				(font
+					(size 1.27 1.27)
+				)
+				(justify left)
+			)
+		)
+		(pin "UCPD_INT" output
+			(at 210.82 99.06 180)
+			(effects
+				(font
+					(size 1.27 1.27)
+				)
+				(justify left)
+			)
+		)
+		(pin "USB_HS_D+" bidirectional
+			(at 210.82 128.27 180)
+			(effects
+				(font
+					(size 1.27 1.27)
+				)
+				(justify left)
+			)
+		)
+		(pin "USB_HS_D-" bidirectional
+			(at 210.82 130.81 180)
+			(effects
+				(font
+					(size 1.27 1.27)
+				)
+				(justify left)
+			)
+		)
+		(pin "UCPD_SCL" input
+			(at 210.82 120.65 180)
+			(effects
+				(font
+					(size 1.27 1.27)
+				)
+				(justify left)
+			)
+		)
+		(pin "UCPD_SDA" bidirectional
+			(at 210.82 123.19 180)
+			(effects
+				(font
+					(size 1.27 1.27)
+				)
+				(justify left)
 			)
 		)
@@
 	)
 	(sheet
-		(at 147.32 35.56)
+		(at 86.36 38.1)
 		(size 82.55 57.15)
 		(exclude_from_sim no)
@@
 		)
 		(property "Sheetname" "MCU"
-			(at 147.32 34.8484 0)
+			(at 86.36 37.3884 0)
 			(effects
 				(font
@@
 		)
 		(property "Sheetfile" "mcu.kicad_sch"
-			(at 147.32 93.2946 0)
+			(at 86.36 95.8346 0)
 			(effects
 				(font
@@
 	)
 	(sheet
-		(at 26.67 29.21)
-		(size 72.39 49.53)
+		(at 210.82 39.37)
+		(size 22.86 41.91)
 		(exclude_from_sim no)
 		(in_bom yes)
@@
 		)
 		(property "Sheetname" "DSP"
-			(at 26.67 28.4984 0)
+			(at 210.82 38.6584 0)
 			(effects
 				(font
@@
 		)
 		(property "Sheetfile" "dsp.kicad_sch"
-			(at 26.67 79.3246 0)
+			(at 210.82 81.8646 0)
 			(effects
 				(font
@@
 			)
 		)
+		(pin "DSP_SDATA_IN0" input
+			(at 210.82 68.58 180)
+			(effects
+				(font
+					(size 1.27 1.27)
+				)
+				(justify left)
+			)
+		)
+		(pin "DSP_LRCLK_OUT0" output
+			(at 210.82 74.93 180)
+			(effects
+				(font
+					(size 1.27 1.27)
+				)
+				(justify left)
+			)
+		)
+		(pin "DSP_BCLK_OUT0" output
+			(at 210.82 72.39 180)
+			(effects
+				(font
+					(size 1.27 1.27)
+				)
+				(justify left)
+			)
+		)
+		(pin "DSP_SDATA_OUT0" output
+			(at 210.82 77.47 180)
+			(effects
+				(font
+					(size 1.27 1.27)
+				)
+				(justify left)
+			)
+		)
+		(pin "DSP_SS" input
+			(at 210.82 48.26 180)
+			(effects
+				(font
+					(size 1.27 1.27)
+				)
+				(justify left)
+			)
+		)
+		(pin "DSP_SCLK" input
+			(at 210.82 50.8 180)
+			(effects
+				(font
+					(size 1.27 1.27)
+				)
+				(justify left)
+			)
+		)
+		(pin "DSP_MOSI" input
+			(at 210.82 53.34 180)
+			(effects
+				(font
+					(size 1.27 1.27)
+				)
+				(justify left)
+			)
+		)
+		(pin "DSP_MISO" output
+			(at 210.82 55.88 180)
+			(effects
+				(font
+					(size 1.27 1.27)
+				)
+				(justify left)
+			)
+		)
+		(pin "DSP_CLKOUT" output
+			(at 210.82 60.96 180)
+			(effects
+				(font
+					(size 1.27 1.27)
+				)
+				(justify left)
+			)
+		)
+		(pin "DSP_LRCLK_IN0" input
+			(at 210.82 66.04 180)
+			(effects
+				(font
+					(size 1.27 1.27)
+				)
+				(justify left)
+			)
+		)
+		(pin "DSP_BCLK_IN0" input
+			(at 210.82 63.5 180)
+			(effects
+				(font
+					(size 1.27 1.27)
+				)
+				(justify left)
+			)
+		)
+		(pin "DSP_RESET" input
+			(at 210.82 43.18 180)
+			(effects
+				(font
+					(size 1.27 1.27)
+				)
+				(justify left)
+			)
+		)

Commit message: Updated schematics.
Other:
- sheet MCU ports: added I2C2_SCL, I2C2_SDA, I2S_CLKIN, SAI_DATA_IN, SAI_DATA_OUT, SAI_FS, SAI_SCK, SPI5_MISO, SPI5_MOSI, SPI5_SCLK, SPI5_SS, UCPD_CC1, UCPD_CC2, UCPD_INT, UCPD_PWR_EN, USB_HS_D+, USB_HS_D-; removed none
Changed lines of the file:
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@@
-			)
-		)
-		(pin "UCPD_ISENSE" input
-			(at 210.82 111.76 180)
-			(effects
-				(font
-					(size 1.27 1.27)
-				)
-				(justify left)
 			)
 		)
@@
 		(pin "UCPD_SDA" bidirectional
 			(at 210.82 123.19 180)
+			(effects
+				(font
+					(size 1.27 1.27)
+				)
+				(justify left)
+			)
+		)
+		(pin "UCPD_ISENSE" output
+			(at 210.82 113.03 180)
 			(effects
 				(font
@@
 	)
 	(sheet
-		(at 48.26 106.68)
-		(size 86.36 69.85)
+		(at 45.72 97.79)
+		(size 36.83 69.85)
 		(exclude_from_sim no)
 		(in_bom yes)
@@
 		)
 		(property "Sheetname" "Power"
-			(at 48.26 105.9684 0)
+			(at 45.72 97.0784 0)
 			(effects
 				(font
@@
 		)
 		(property "Sheetfile" "power.kicad_sch"
-			(at 48.26 177.1146 0)
+			(at 45.72 168.2246 0)
 			(effects
 				(font
@@
 	)
 	(sheet
-		(at 86.36 38.1)
-		(size 82.55 57.15)
+		(at 107.95 39.37)
+		(size 82.55 96.52)
 		(exclude_from_sim no)
 		(in_bom yes)
@@
 		)
 		(property "Sheetname" "MCU"
-			(at 86.36 37.3884 0)
+			(at 107.95 38.6584 0)
 			(effects
 				(font
@@
 		)
 		(property "Sheetfile" "mcu.kicad_sch"
-			(at 86.36 95.8346 0)
+			(at 107.95 136.4746 0)
 			(effects
 				(font
@@
 				)
 				(justify left top)
+			)
+		)
+		(pin "SAI_DATA_OUT" input
+			(at 190.5 68.58 0)
+			(effects
+				(font
+					(size 1.27 1.27)
+				)
+				(justify right)
+			)
+		)
+		(pin "SAI_SCK" input
+			(at 190.5 72.39 0)
+			(effects
+				(font
+					(size 1.27 1.27)
+				)
+				(justify right)
+			)
+		)
+		(pin "UCPD_CC2" bidirectional
+			(at 190.5 106.68 0)
+			(effects
+				(font
+					(size 1.27 1.27)
+				)
+				(justify right)
+			)
+		)
+		(pin "UCPD_PWR_EN" output
+			(at 190.5 96.52 0)
+			(effects
+				(font
+					(size 1.27 1.27)
+				)
+				(justify right)
+			)
+		)
+		(pin "UCPD_CC1" bidirectional
+			(at 190.5 104.14 0)
+			(effects
+				(font
+					(size 1.27 1.27)
+				)
+				(justify right)
+			)
+		)
+		(pin "SAI_FS" input
+			(at 190.5 74.93 0)
+			(effects
+				(font
+					(size 1.27 1.27)
+				)
+				(justify right)
+			)
+		)
+		(pin "I2S_CLKIN" input
+			(at 190.5 60.96 0)
+			(effects
+				(font
+					(size 1.27 1.27)
+				)
+				(justify right)
+			)
+		)
+		(pin "USB_HS_D+" bidirectional
+			(at 190.5 128.27 0)
+			(effects
+				(font
+					(size 1.27 1.27)
+				)
+				(justify right)
+			)
+		)
+		(pin "SAI_DATA_IN" input
+			(at 190.5 77.47 0)
+			(effects
+				(font
+					(size 1.27 1.27)
+				)
+				(justify right)
+			)
+		)
+		(pin "USB_HS_D-" bidirectional
+			(at 190.5 130.81 0)
+			(effects
+				(font
+					(size 1.27 1.27)
+				)
+				(justify right)
+			)
+		)
+		(pin "UCPD_INT" input
+			(at 190.5 99.06 0)
+			(effects
+				(font
+					(size 1.27 1.27)
+				)
+				(justify right)
+			)
+		)
+		(pin "SPI5_SS" output
+			(at 190.5 48.26 0)
+			(effects
+				(font
+					(size 1.27 1.27)
+				)
+				(justify right)
+			)
+		)
+		(pin "SPI5_MOSI" output
+			(at 190.5 53.34 0)
+			(effects
+				(font
+					(size 1.27 1.27)
+				)
+				(justify right)
+			)
+		)
+		(pin "SPI5_SCLK" output
+			(at 190.5 50.8 0)
+			(effects
+				(font
+					(size 1.27 1.27)
+				)
+				(justify right)
+			)
+		)
+		(pin "SPI5_MISO" input
+			(at 190.5 55.88 0)
+			(effects
+				(font
+					(size 1.27 1.27)
+				)
+				(justify right)
+			)
+		)
+		(pin "I2C2_SDA" bidirectional
+			(at 190.5 123.19 0)
+			(effects
+				(font
+					(size 1.27 1.27)
+				)
+				(justify right)
+			)
+		)
+		(pin "I2C2_SCL" output
+			(at 190.5 120.65 0)
+			(effects
+				(font
+					(size 1.27 1.27)
+				)
+				(justify right)
 			)
 		)
@@
 	(sheet
 		(at 210.82 39.37)
-		(size 22.86 41.91)
+		(size 48.26 41.91)
 		(exclude_from_sim no)
 		(in_bom yes)

Commit message: Updated schematics.
Other:
- sheet MCU ports: added DSP_RESET; removed none
Changed lines of the file:
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@@
 	(generator_version "9.0")
 	(paper "A4")
+	(wire
+		(pts
+			(xy 190.5 104.14) (xy 210.82 104.14)
+		)
+		(stroke
+			(width 0)
+			(type default)
+		)
+	)
+	(wire
+		(pts
+			(xy 190.5 96.52) (xy 210.82 96.52)
+		)
+		(stroke
+			(width 0)
+			(type default)
+		)
+	)
+	(wire
+		(pts
+			(xy 190.5 106.68) (xy 210.82 106.68)
+		)
+		(stroke
+			(width 0)
+			(type default)
+		)
+	)
+	(wire
+		(pts
+			(xy 190.5 55.88) (xy 210.82 55.88)
+		)
+		(stroke
+			(width 0)
+			(type default)
+		)
+	)
+	(wire
+		(pts
+			(xy 190.5 123.19) (xy 210.82 123.19)
+		)
+		(stroke
+			(width 0)
+			(type default)
+		)
+	)
+	(wire
+		(pts
+			(xy 190.5 72.39) (xy 210.82 72.39)
+		)
+		(stroke
+			(width 0)
+			(type default)
+		)
+	)
+	(wire
+		(pts
+			(xy 190.5 74.93) (xy 210.82 74.93)
+		)
+		(stroke
+			(width 0)
+			(type default)
+		)
+	)
+	(wire
+		(pts
+			(xy 190.5 48.26) (xy 210.82 48.26)
+		)
+		(stroke
+			(width 0)
+			(type default)
+		)
+	)
+	(wire
+		(pts
+			(xy 190.5 128.27) (xy 210.82 128.27)
+		)
+		(stroke
+			(width 0)
+			(type default)
+		)
+	)
+	(wire
+		(pts
+			(xy 190.5 130.81) (xy 210.82 130.81)
+		)
+		(stroke
+			(width 0)
+			(type default)
+		)
+	)
+	(wire
+		(pts
+			(xy 190.5 60.96) (xy 210.82 60.96)
+		)
+		(stroke
+			(width 0)
+			(type default)
+		)
+	)
+	(wire
+		(pts
+			(xy 190.5 50.8) (xy 210.82 50.8)
+		)
+		(stroke
+			(width 0)
+			(type default)
+		)
+	)
+	(wire
+		(pts
+			(xy 190.5 120.65) (xy 210.82 120.65)
+		)
+		(stroke
+			(width 0)
+			(type default)
+		)
+	)
+	(wire
+		(pts
+			(xy 190.5 53.34) (xy 210.82 53.34)
+		)
+		(stroke
+			(width 0)
+			(type default)
+		)
+	)
+	(wire
+		(pts
+			(xy 190.5 43.18) (xy 210.82 43.18)
+		)
+		(stroke
+			(width 0)
+			(type default)
+		)
+	)
+	(wire
+		(pts
+			(xy 190.5 99.06) (xy 210.82 99.06)
+		)
+		(stroke
+			(width 0)
+			(type default)
+		)
+	)
+	(wire
+		(pts
+			(xy 190.5 77.47) (xy 210.82 77.47)
+		)
+		(stroke
+			(width 0)
+			(type default)
+		)
+	)
+	(wire
+		(pts
+			(xy 190.5 68.58) (xy 210.82 68.58)
+		)
+		(stroke
+			(width 0)
+			(type default)
+		)
+	)
 	(sheet
 		(at 210.82 91.44)
@@
 			)
 		)
-		(pin "SAI_DATA_OUT" input
+		(pin "SAI_DATA_OUT" output
 			(at 190.5 68.58 0)
 			(effects
@@
 		(pin "I2C2_SCL" output
 			(at 190.5 120.65 0)
+			(effects
+				(font
+					(size 1.27 1.27)
+				)
+				(justify right)
+			)
+		)
+		(pin "DSP_RESET" output
+			(at 190.5 43.18 0)
 			(effects
 				(font
@@
 	(sheet
 		(at 210.82 39.37)
-		(size 48.26 41.91)
+		(size 24.13 41.91)
 		(exclude_from_sim no)
 		(in_bom yes)

Commit message: Updated schematics.
Other:
- sheet MCU ports: added UCPD_ISENSE; removed none

Commit message: Modified wiring between ICs.
Other:
- sheet MCU ports: added SAI1A_DATA_IN, SAI1A_FS, SAI1A_SCK, SAI1B_DATA_IN, SAI2A_DATA_OUT, SAI2A_FS, SAI2A_SCK; removed SAI_DATA_IN, SAI_DATA_OUT, SAI_FS, SAI_SCK
Changed lines of the file:
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@@
+	(wire
+		(pts
+			(xy 152.4 72.39) (xy 172.72 72.39)
+		)
+		(stroke
+			(width 0)
+			(type default)
+		)
+	)
 	(wire
 		(pts
@@
 	(wire
 		(pts
+			(xy 152.4 86.36) (xy 172.72 86.36)
+		)
+		(stroke
+			(width 0)
+			(type default)
+		)
+	)
+	(wire
+		(pts
 			(xy 152.4 69.85) (xy 172.72 69.85)
 		)
@@
 	(wire
 		(pts
+			(xy 152.4 74.93) (xy 172.72 74.93)
+		)
+		(stroke
+			(width 0)
+			(type default)
+		)
+	)
+	(wire
+		(pts
+			(xy 152.4 109.22) (xy 172.72 109.22)
+		)
+		(stroke
+			(width 0)
+			(type default)
+		)
+	)
+	(wire
+		(pts
+			(xy 152.4 58.42) (xy 172.72 58.42)
+		)
+		(stroke
+			(width 0)
+			(type default)
+		)
+	)
+	(wire
+		(pts
 			(xy 152.4 77.47) (xy 172.72 77.47)
 		)
@@
 	(wire
 		(pts
-			(xy 152.4 109.22) (xy 172.72 109.22)
-		)
-		(stroke
-			(width 0)
-			(type default)
-		)
-	)
-	(wire
-		(pts
-			(xy 152.4 58.42) (xy 172.72 58.42)
-		)
-		(stroke
-			(width 0)
-			(type default)
-		)
-	)
-	(wire
-		(pts
 			(xy 152.4 81.28) (xy 172.72 81.28)
 		)
@@
 		(pts
 			(xy 152.4 54.61) (xy 172.72 54.61)
-		)
-		(stroke
-			(width 0)
-			(type default)
-		)
-	)
-	(wire
-		(pts
-			(xy 152.4 86.36) (xy 172.72 86.36)
 		)
 		(stroke
@@
 			)
 		)
-		(pin "SAI_DATA_OUT" output
-			(at 152.4 77.47 0)
-			(effects
-				(font
-					(size 1.27 1.27)
-				)
-				(justify right)
-			)
-		)
-		(pin "SAI_SCK" input
+		(pin "SAI1A_DATA_IN" input
+			(at 152.4 86.36 0)
+			(effects
+				(font
+					(size 1.27 1.27)
+				)
+				(justify right)
+			)
+		)
+		(pin "SAI1A_SCK" input
 			(at 152.4 81.28 0)
 			(effects
@@
 			)
 		)
-		(pin "SAI_FS" input
+		(pin "SAI1A_FS" input
 			(at 152.4 83.82 0)
 			(effects
@@
 			)
 		)
-		(pin "SAI_DATA_IN" input
-			(at 152.4 86.36 0)
+		(pin "SAI1B_DATA_IN" input
+			(at 152.4 88.9 0)
 			(effects
 				(font
@@
 		(pin "UCPD_ISENSE" input
 			(at 152.4 121.92 0)
+			(effects
+				(font
+					(size 1.27 1.27)
+				)
+				(justify right)
+			)
+		)
+		(pin "SAI2A_FS" input
+			(at 152.4 74.93 0)
+			(effects
+				(font
+					(size 1.27 1.27)
+				)
+				(justify right)
+			)
+		)
+		(pin "SAI2A_SCK" input
+			(at 152.4 72.39 0)
+			(effects
+				(font
+					(size 1.27 1.27)
+				)
+				(justify right)
+			)
+		)
+		(pin "SAI2A_DATA_OUT" output
+			(at 152.4 77.47 0)
 			(effects
 				(font
@@
 			)
 		)
-		(pin "DSP_LRCLK_IN0" input
+		(pin "DSP_LRCLK_IN0" output
 			(at 172.72 74.93 180)
 			(effects
@@
 			)
 		)
-		(pin "DSP_BCLK_IN0" input
+		(pin "DSP_BCLK_IN0" output
 			(at 172.72 72.39 180)
 			(effects

Commit message: Improved some routes.
Other:
- sheet MCU ports: added none; removed SAI1B_DATA_IN
Changed lines of the file:
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@@
-			)
-		)
-		(pin "SAI1B_DATA_IN" input
-			(at 152.4 88.9 0)
-			(effects
-				(font
-					(size 1.27 1.27)
-				)
-				(justify right)
 			)
 		)
