File: KiCad/OTO_NO_ITA/power.kicad_sch (KiCad schematic)
At the start: 0 parts

Commit message: Updated schematics.
Parts:
- added C32, C34, C36: 4.7uF, Capacitor_SMD:C_0603_1608Metric, symbol Device:C
- added C33, C35, C37: 1uF, Capacitor_SMD:C_0603_1608Metric, symbol Device:C
- added U10: AP2127N-1.8TRG1, Package_TO_SOT_SMD:SOT-23, symbol Regulator_Linear:AP2127N-1.8
- added U9: AP7361EA-33E-13, Package_TO_SOT_SMD:SOT-223-3_TabPin2, symbol Regulator_Linear:AP7361C-18E
Connections:
- new net 1V8: C35.1, C37.1, U10.2 (VO)
- new net 3V3: C34.1, C36.1, U9.3 (VO)
- new net 5V: C32.1, C33.1, U10.3 (VI), U9.1 (VI)
- new net GND: C32.2, C33.2, C34.2, C35.2, C36.2, C37.2, U10.1 (GND), U9.2 (GND)

Commit message: Updated schematics.
Other:
- moved on the sheet: C32, C33, C34, C35, C36, C37, U10, U9

Commit message: Updated schematics.
Parts:
- renumbered C32 to C59, C34 to C60, C36 to C61, C33 to C62, C35 to C63, C37 to C64, U9 to U5, U10 to U6
Changed lines of the file:
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@@
 		(dnp no)
 		(fields_autoplaced yes)
-		(property "Reference" "#PWR044"
+		(property "Reference" "#PWR067"
 			(at 160.02 99.06 0)
 			(effects
@@
 			(project "OTO_NO_ITA"
 				(path "/9c594957-fd6c-4305-bab8-fba79a4c5d5c/d3891a31-cd10-4fb1-a9a6-73758f166e5e"
-					(reference "#PWR044")
+					(reference "#PWR067")
 					(unit 1)
 				)
@@
 		(dnp no)
 		(fields_autoplaced yes)
-		(property "Reference" "#PWR043"
+		(property "Reference" "#PWR064"
 			(at 160.02 71.755 0)
 			(effects
@@
 			(project "OTO_NO_ITA"
 				(path "/9c594957-fd6c-4305-bab8-fba79a4c5d5c/d3891a31-cd10-4fb1-a9a6-73758f166e5e"
-					(reference "#PWR043")
+					(reference "#PWR064")
 					(unit 1)
 				)
@@
 		(on_board yes)
 		(dnp no)
-		(property "Reference" "C36"
+		(property "Reference" "C61"
 			(at 161.29 74.295 0)
 			(effects
@@
 			(project "OTO_NO_ITA"
 				(path "/9c594957-fd6c-4305-bab8-fba79a4c5d5c/d3891a31-cd10-4fb1-a9a6-73758f166e5e"
-					(reference "C36")
+					(reference "C61")
 					(unit 1)
 				)
@@
 		(on_board yes)
 		(dnp no)
-		(property "Reference" "U9"
+		(property "Reference" "U5"
 			(at 138.43 65.405 0)
 			(effects
@@
 			(project "OTO_NO_ITA"
 				(path "/9c594957-fd6c-4305-bab8-fba79a4c5d5c/d3891a31-cd10-4fb1-a9a6-73758f166e5e"
-					(reference "U9")
+					(reference "U5")
 					(unit 1)
 				)
@@
 		(on_board yes)
 		(dnp no)
-		(property "Reference" "C33"
+		(property "Reference" "C62"
 			(at 130.81 101.6 0)
 			(effects
@@
 			(project "OTO_NO_ITA"
 				(path "/9c594957-fd6c-4305-bab8-fba79a4c5d5c/d3891a31-cd10-4fb1-a9a6-73758f166e5e"
-					(reference "C33")
+					(reference "C62")
 					(unit 1)
 				)
@@
 		(on_board yes)
 		(dnp no)
-		(property "Reference" "C32"
+		(property "Reference" "C59"
 			(at 130.81 74.295 0)
 			(effects
@@
 			(project "OTO_NO_ITA"
 				(path "/9c594957-fd6c-4305-bab8-fba79a4c5d5c/d3891a31-cd10-4fb1-a9a6-73758f166e5e"
-					(reference "C32")
+					(reference "C59")
 					(unit 1)
 				)
@@
 		(dnp no)
 		(fields_autoplaced yes)
-		(property "Reference" "#PWR039"
+		(property "Reference" "#PWR063"
 			(at 129.54 71.755 0)
 			(effects
@@
 			(project "OTO_NO_ITA"
 				(path "/9c594957-fd6c-4305-bab8-fba79a4c5d5c/d3891a31-cd10-4fb1-a9a6-73758f166e5e"
-					(reference "#PWR039")
+					(reference "#PWR063")
 					(unit 1)
 				)
@@
 		(on_board yes)
 		(dnp no)
-		(property "Reference" "#PWR042"
+		(property "Reference" "#PWR068"
 			(at 142.24 116.84 0)
 			(effects
@@
 			(project "OTO_NO_ITA"
 				(path "/9c594957-fd6c-4305-bab8-fba79a4c5d5c/d3891a31-cd10-4fb1-a9a6-73758f166e5e"
-					(reference "#PWR042")
+					(reference "#PWR068")
 					(unit 1)
 				)
@@
 		(on_board yes)
 		(dnp no)
-		(property "Reference" "C37"
+		(property "Reference" "C64"
 			(at 161.29 101.6 0)
 			(effects
@@
 			(project "OTO_NO_ITA"
 				(path "/9c594957-fd6c-4305-bab8-fba79a4c5d5c/d3891a31-cd10-4fb1-a9a6-73758f166e5e"
-					(reference "C37")
+					(reference "C64")
 					(unit 1)
 				)
@@
 		(on_board yes)
 		(dnp no)
-		(property "Reference" "C34"
+		(property "Reference" "C60"
 			(at 153.67 74.295 0)
 			(effects
@@
 			(project "OTO_NO_ITA"
 				(path "/9c594957-fd6c-4305-bab8-fba79a4c5d5c/d3891a31-cd10-4fb1-a9a6-73758f166e5e"
-					(reference "C34")
+					(reference "C60")
 					(unit 1)
 				)
@@
 		(dnp no)
 		(fields_autoplaced yes)
-		(property "Reference" "#PWR040"
+		(property "Reference" "#PWR066"
 			(at 129.54 99.06 0)
 			(effects
@@
 			(project "OTO_NO_ITA"
 				(path "/9c594957-fd6c-4305-bab8-fba79a4c5d5c/d3891a31-cd10-4fb1-a9a6-73758f166e5e"
-					(reference "#PWR040")
+					(reference "#PWR066")
 					(unit 1)
 				)
@@
 		(dnp no)
 		(fields_autoplaced yes)
-		(property "Reference" "U10"
+		(property "Reference" "U6"
 			(at 142.24 91.44 0)
 			(effects
@@
 			(project "OTO_NO_ITA"
 				(path "/9c594957-fd6c-4305-bab8-fba79a4c5d5c/d3891a31-cd10-4fb1-a9a6-73758f166e5e"
-					(reference "U10")
+					(reference "U6")
 					(unit 1)
 				)
@@
 		(on_board yes)
 		(dnp no)
-		(property "Reference" "#PWR041"
+		(property "Reference" "#PWR065"
 			(at 142.24 89.535 0)
 			(effects
@@
 			(project "OTO_NO_ITA"
 				(path "/9c594957-fd6c-4305-bab8-fba79a4c5d5c/d3891a31-cd10-4fb1-a9a6-73758f166e5e"
-					(reference "#PWR041")
+					(reference "#PWR065")
 					(unit 1)
 				)
@@
 		(on_board yes)
 		(dnp no)
-		(property "Reference" "C35"
+		(property "Reference" "C63"
 			(at 153.67 101.6 0)
 			(effects
@@
 			(project "OTO_NO_ITA"
 				(path "/9c594957-fd6c-4305-bab8-fba79a4c5d5c/d3891a31-cd10-4fb1-a9a6-73758f166e5e"
-					(reference "C35")
-					(unit 1)
-				)
+					(reference "C63")
+					(unit 1)
+				)

Commit message: Re-annotation.
Parts:
- renumbered C59 to C62, C60 to C63, C61 to C64, C62 to C65, C63 to C66, C64 to C67
Changed lines of the file:
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@@
 		(dnp no)
 		(fields_autoplaced yes)
-		(property "Reference" "#PWR067"
+		(property "Reference" "#PWR078"
 			(at 160.02 99.06 0)
 			(effects
@@
 			(project "OTO_NO_ITA"
 				(path "/9c594957-fd6c-4305-bab8-fba79a4c5d5c/d3891a31-cd10-4fb1-a9a6-73758f166e5e"
-					(reference "#PWR067")
+					(reference "#PWR078")
 					(unit 1)
 				)
@@
 		(dnp no)
 		(fields_autoplaced yes)
-		(property "Reference" "#PWR064"
+		(property "Reference" "#PWR075"
 			(at 160.02 71.755 0)
 			(effects
@@
 			(project "OTO_NO_ITA"
 				(path "/9c594957-fd6c-4305-bab8-fba79a4c5d5c/d3891a31-cd10-4fb1-a9a6-73758f166e5e"
-					(reference "#PWR064")
+					(reference "#PWR075")
 					(unit 1)
 				)
@@
 		(on_board yes)
 		(dnp no)
-		(property "Reference" "C61"
+		(property "Reference" "C64"
 			(at 161.29 74.295 0)
 			(effects
@@
 			(project "OTO_NO_ITA"
 				(path "/9c594957-fd6c-4305-bab8-fba79a4c5d5c/d3891a31-cd10-4fb1-a9a6-73758f166e5e"
-					(reference "C61")
+					(reference "C64")
 					(unit 1)
 				)
@@
 		(on_board yes)
 		(dnp no)
-		(property "Reference" "C62"
+		(property "Reference" "C65"
 			(at 130.81 101.6 0)
 			(effects
@@
 			(project "OTO_NO_ITA"
 				(path "/9c594957-fd6c-4305-bab8-fba79a4c5d5c/d3891a31-cd10-4fb1-a9a6-73758f166e5e"
-					(reference "C62")
+					(reference "C65")
 					(unit 1)
 				)
@@
 		(on_board yes)
 		(dnp no)
-		(property "Reference" "C59"
+		(property "Reference" "C62"
 			(at 130.81 74.295 0)
 			(effects
@@
 			(project "OTO_NO_ITA"
 				(path "/9c594957-fd6c-4305-bab8-fba79a4c5d5c/d3891a31-cd10-4fb1-a9a6-73758f166e5e"
-					(reference "C59")
+					(reference "C62")
 					(unit 1)
 				)
@@
 		(dnp no)
 		(fields_autoplaced yes)
-		(property "Reference" "#PWR063"
+		(property "Reference" "#PWR074"
 			(at 129.54 71.755 0)
 			(effects
@@
 			(project "OTO_NO_ITA"
 				(path "/9c594957-fd6c-4305-bab8-fba79a4c5d5c/d3891a31-cd10-4fb1-a9a6-73758f166e5e"
-					(reference "#PWR063")
+					(reference "#PWR074")
 					(unit 1)
 				)
@@
 		(on_board yes)
 		(dnp no)
-		(property "Reference" "#PWR068"
+		(property "Reference" "#PWR079"
 			(at 142.24 116.84 0)
 			(effects
@@
 			(project "OTO_NO_ITA"
 				(path "/9c594957-fd6c-4305-bab8-fba79a4c5d5c/d3891a31-cd10-4fb1-a9a6-73758f166e5e"
-					(reference "#PWR068")
+					(reference "#PWR079")
 					(unit 1)
 				)
@@
 		(on_board yes)
 		(dnp no)
-		(property "Reference" "C64"
+		(property "Reference" "C67"
 			(at 161.29 101.6 0)
 			(effects
@@
 			(project "OTO_NO_ITA"
 				(path "/9c594957-fd6c-4305-bab8-fba79a4c5d5c/d3891a31-cd10-4fb1-a9a6-73758f166e5e"
-					(reference "C64")
+					(reference "C67")
 					(unit 1)
 				)
@@
 		(on_board yes)
 		(dnp no)
-		(property "Reference" "C60"
+		(property "Reference" "C63"
 			(at 153.67 74.295 0)
 			(effects
@@
 			(project "OTO_NO_ITA"
 				(path "/9c594957-fd6c-4305-bab8-fba79a4c5d5c/d3891a31-cd10-4fb1-a9a6-73758f166e5e"
-					(reference "C60")
+					(reference "C63")
 					(unit 1)
 				)
@@
 		(dnp no)
 		(fields_autoplaced yes)
-		(property "Reference" "#PWR066"
+		(property "Reference" "#PWR077"
 			(at 129.54 99.06 0)
 			(effects
@@
 			(project "OTO_NO_ITA"
 				(path "/9c594957-fd6c-4305-bab8-fba79a4c5d5c/d3891a31-cd10-4fb1-a9a6-73758f166e5e"
-					(reference "#PWR066")
+					(reference "#PWR077")
 					(unit 1)
 				)
@@
 		(on_board yes)
 		(dnp no)
-		(property "Reference" "#PWR065"
+		(property "Reference" "#PWR076"
 			(at 142.24 89.535 0)
 			(effects
@@
 			(project "OTO_NO_ITA"
 				(path "/9c594957-fd6c-4305-bab8-fba79a4c5d5c/d3891a31-cd10-4fb1-a9a6-73758f166e5e"
-					(reference "#PWR065")
+					(reference "#PWR076")
 					(unit 1)
 				)
@@
 		(on_board yes)
 		(dnp no)
-		(property "Reference" "C63"
+		(property "Reference" "C66"
 			(at 153.67 101.6 0)
 			(effects
@@
 			(project "OTO_NO_ITA"
 				(path "/9c594957-fd6c-4305-bab8-fba79a4c5d5c/d3891a31-cd10-4fb1-a9a6-73758f166e5e"
-					(reference "C63")
-					(unit 1)
-				)
+					(reference "C66")
+					(unit 1)
+				)

Commit message: Fixed some mistakes.
switched 5V and 5V_UCPD.
switched VREFP and VREFM.
Connections:
- net 5V renamed 5V_UCPD
Changed lines of the file:
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@@
 		(on_board yes)
 		(dnp no)
-		(fields_autoplaced yes)
 		(property "Reference" "#PWR074"
 			(at 129.54 71.755 0)
@@
 			)
 		)
-		(property "Value" "5V"
-			(at 129.54 62.865 0)
-			(effects
-				(font
-					(size 1.27 1.27)
-				)
+		(property "Value" "5V_UCPD"
+			(at 125.476 63.5 0)
+			(effects
+				(font
+					(size 1.27 1.27)
+				)
+				(justify left)
 			)
 		)
@@
 		(on_board yes)
 		(dnp no)
-		(fields_autoplaced yes)
 		(property "Reference" "#PWR077"
 			(at 129.54 99.06 0)
@@
 			)
 		)
-		(property "Value" "5V"
-			(at 129.54 90.805 0)
-			(effects
-				(font
-					(size 1.27 1.27)
-				)
-			)
-		)
+		(property "Value" "5V_UCPD"
+			(at 125.476 90.932 0)
+			(effects
+				(font
+					(size 1.27 1.27)
+				)
+				(justify left)
+			)
+		)
