File: KiCad/OTO_NO_TE/OTO_NO_TE.kicad_pcb (KiCad board)
At the start: 4 copper layers, 114.3 x 85 mm, 87 parts, among them J1 Conn_01x06, J2 Conn_01x06, J3 Conn_01x06, U1 DRV5056A3QDBZR, U10 DRV5056A3QDBZR, U11 DRV5056A3QDBZR, U2 DRV5056A3QDBZR, U3 DRV5056A3QDBZR, U4 DRV5056A3QDBZR, U5 DRV5056A3QDBZR, U6 DRV5056A3QDBZR, U7 DRV5056A3QDBZR, U8 CD74HC4067M, U9 DRV5056A3QDBZR

Commit message: アナログマルチプレクサの配線修正と部品番号を整理
Parts:
- renumbered RV4 to RV10, RV8 to RV11, RV5 to RV2, RV9 to RV3, RV3 to RV4, RV7 to RV5, RV11 to RV6, RV2 to RV7, RV6 to RV8, RV10 to RV9
Connections:
- RV10 pad 2: /R1 -> /R3
- RV11 pad 2: /R3 -> /R4
- RV2 pad 2: /L2 -> /L1
- RV3 pad 2: /L4 -> /L2
- RV4 pad 2: /L1 -> /L3
- RV5 pad 2: /L3 -> /L4
- RV6 pad 2: /R4 -> /L5
- RV8 pad 2: /R2 -> /R1
- RV9 pad 2: /L5 -> /R2
Routing:
- net /L5: track 108.2 -> 43.8 mm
- net /R4: track 38.4 -> 79.5 mm
- net /R1: track 63.6 -> 94.4 mm
- net /L4: track 51.6 -> 21.1 mm
- net /L1: track 12.3 -> 33.1 mm, vias 1 -> 0
- net /L2: track 34.7 -> 53.5 mm
- net /R3: track 77.3 -> 58.5 mm
- net /R2: track 97.2 -> 113.4 mm
- net /L3: track 22.3 -> 24.9 mm, vias 0 -> 1
- net /R0: track 70.7 -> 73.0 mm
- net Net-(J1-Pin_5): track 22.7 -> 23.3 mm
