File: KiCad/OTO_NO_TE/OTO_NO_TE.kicad_sch (KiCad schematic)
At the start: 57 parts, among them J1 Conn_01x06, J2 Conn_01x06, J3 Conn_01x06, U1 DRV5056A3QDBZR, U10 DRV5056A3QDBZR, U11 DRV5056A3QDBZR, U2 DRV5056A3QDBZR, U3 DRV5056A3QDBZR, U4 DRV5056A3QDBZR, U5 DRV5056A3QDBZR, U6 DRV5056A3QDBZR, U7 DRV5056A3QDBZR, U8 CD74HC4067M, U9 DRV5056A3QDBZR

Commit message: アナログマルチプレクサの配線修正と部品番号を整理
Parts:
- renumbered RV4 to RV10, RV8 to RV11, RV5 to RV2, RV9 to RV3, RV3 to RV4, RV7 to RV5, RV11 to RV6, RV2 to RV7, RV6 to RV8, RV10 to RV9
Connections:
- net L1: now also RV2.2; no longer RV4.2
- net L2: now also RV3.2; no longer RV2.2
- net L3: now also RV4.2; no longer RV5.2
- net L4: now also RV5.2; no longer RV3.2
- net L5: now also RV6.2; no longer RV9.2
- net R1: now also RV8.2; no longer RV10.2
- net R2: now also RV9.2; no longer RV8.2
- net R3: now also RV10.2; no longer RV11.2
- net R4: now also RV11.2; no longer RV6.2
Other:
- moved on the sheet: RV1, RV10, RV11, RV12, RV2, RV3, RV4, RV5, RV6, RV7, RV8, RV9
